File: zmk-g915.kicad_pcb (KiCad board)
At the start: 2 copper layers, 284.7 x 94.2 mm, 203 parts, among them J1 JST-4-pin, J3 Prog_conn, J4 TYPE-C-31-M12_13, J5 Tag connect TC2030-CTX, SW2 Reset Switch, U1 BQ24074RGTR, U3 nRF52840-QIAA-R/nRF52833-QIAA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, U4 TPD4E05U06DQAR, Y1 32MHz, Y2 32.768kHz

Commit message: Layout start. Add symbols to proj lib
Parts:
- removed G***: LOGO, keyboard:keyboard-name-silkscreen
- removed G***: LOGO, keyboard:logo-soldermask
- removed G***: LOGO, keyboard:creator_logo
- removed R18: 10k, keyboard:R_0402_1005Metric
- removed S4: ~, keyboard:ZMK_logo
- removed SW2: Reset Switch, keyboard:RST_SW
- added C100: 100nF, Capacitor_SMD:C_0402_1005Metric, F.Cu at (262.8, 134.5)
- added C101: 100nF, Capacitor_SMD:C_0402_1005Metric, F.Cu at (281.9, 134.5)
- added C102: 100nF, Capacitor_SMD:C_0402_1005Metric, F.Cu at (317.6, 134.5)
- added C103: 100nF, Capacitor_SMD:C_0402_1005Metric, F.Cu at (379.0, 134.5)
- added C104: 100nF, Capacitor_SMD:C_0402_1005Metric, F.Cu at (423.8, 134.5)
- added C105: 100nF, Capacitor_SMD:C_0402_1005Metric, F.Cu at (442.8, 134.5)
- added C106: 100nF, Capacitor_SMD:C_0402_1005Metric, F.Cu at (461.9, 134.5)
- added C107: 100nF, Capacitor_SMD:C_0402_1005Metric, F.Cu at (480.9, 144.0)
- added C108: 100nF, Capacitor_SMD:C_0402_1005Metric, F.Cu at (43.6, 153.6)
- added C109: 100nF, Capacitor_SMD:C_0402_1005Metric, F.Cu at (72.3, 153.6)
- added C110: 100nF, Capacitor_SMD:C_0402_1005Metric, F.Cu at (98.5, 153.6)
- added C111: 100nF, Capacitor_SMD:C_0402_1005Metric, F.Cu at (122.3, 153.6)
- added C112: 100nF, Capacitor_SMD:C_0402_1005Metric, F.Cu at (189.0, 153.6)
- added C113: 100nF, Capacitor_SMD:C_0402_1005Metric, F.Cu at (255.7, 153.6)
- added C114: 100nF, Capacitor_SMD:C_0402_1005Metric, F.Cu at (279.5, 153.6)
- added C115: 100nF, Capacitor_SMD:C_0402_1005Metric, F.Cu at (303.3, 153.6)
- added C116: 100nF, Capacitor_SMD:C_0402_1005Metric, F.Cu at (329.5, 153.6)
- added C117: 100nF, Capacitor_SMD:C_0402_1005Metric, F.Cu at (360.0, 153.6)
- added C118: 100nF, Capacitor_SMD:C_0402_1005Metric, F.Cu at (379.0, 153.6)
- added C119: 100nF, Capacitor_SMD:C_0402_1005Metric, F.Cu at (398.1, 153.6)
- added C120: 100nF, Capacitor_SMD:C_0402_1005Metric, F.Cu at (433.3, 153.6)
- added C121: 100nF, Capacitor_SMD:C_0402_1005Metric, F.Cu at (461.9, 153.6)
- added C122: 4u7F, keyboard:C_0805_2012Metric, F.Cu at (-88.1, -64.4)
- added C123: 8pF, keyboard:C_0402_1005Metric, F.Cu at (-97.5, -64.9)
- added C124: 8pF, keyboard:C_0402_1005Metric, F.Cu at (-97.5, -63.0)
- added C125: 1uF, keyboard:C_0603_1608Metric, F.Cu at (-71.6, -60.0)
- added C126: 100nF, keyboard:C_0402_1005Metric, F.Cu at (-97.5, -61.0)
- added C127: 1uF, keyboard:C_0603_1608Metric, F.Cu at (-71.6, -57.5)
- added C128: 100nF, keyboard:C_0402_1005Metric, F.Cu at (-97.5, -59.0)
- added C129: 8pF, keyboard:C_0402_1005Metric, F.Cu at (-97.5, -57.1)
- added C130: 8pF, keyboard:C_0402_1005Metric, F.Cu at (-94.6, -64.9)
- added C131: 100nF, keyboard:C_0402_1005Metric, F.Cu at (-94.6, -63.0)
- added C132: 820pF, keyboard:C_0402_1005Metric, F.Cu at (-94.6, -61.0)
- added C133: 100pF, keyboard:C_0402_1005Metric, F.Cu at (-94.6, -59.0)
- added C134: DNP, keyboard:C_0402_1005Metric, F.Cu at (-94.6, -57.1)
- added C135: 100nF, keyboard:C_0402_1005Metric, F.Cu at (-91.7, -64.9)
- added C136: 100nF, keyboard:C_0402_1005Metric, F.Cu at (-91.7, -63.0)
- added C137: 4u7F, keyboard:C_0805_2012Metric, F.Cu at (-88.1, -61.4)
- added C138: 1pF, keyboard:C_0402_1005Metric, F.Cu at (-91.7, -61.0)
- added C139: 4u7F, keyboard:C_0805_2012Metric, F.Cu at (-88.1, -58.4)
- added C140: 1.2pF, keyboard:C_0402_1005Metric, F.Cu at (-91.7, -59.0)
- added C141: 1uF, keyboard:C_0603_1608Metric, F.Cu at (-43.5, -27.9)
- added C142: 4u7F, keyboard:C_0805_2012Metric, F.Cu at (-47.3, -30.6)
- added C143: 100nF, keyboard:C_0402_1005Metric, F.Cu at (-44.0, -25.6)
- added C15: 100nF, Capacitor_SMD:C_0402_1005Metric, F.Cu at (207.3, 53.5)
- added C18: 100nF, Capacitor_SMD:C_0402_1005Metric, F.Cu at (277.1, 53.5)
- added C19: 100nF, Capacitor_SMD:C_0402_1005Metric, F.Cu at (296.2, 53.5)
- added C28: 100nF, Capacitor_SMD:C_0402_1005Metric, F.Cu at (481.0, 53.5)
- added C29: 100nF, Capacitor_SMD:C_0402_1005Metric, F.Cu at (43.6, 77.4)
- added C3: 100nF, Capacitor_SMD:C_0402_1005Metric, F.Cu at (137.4, 34.5)
- added C30: 100nF, Capacitor_SMD:C_0402_1005Metric, F.Cu at (67.6, 77.4)
- added C31: 100nF, Capacitor_SMD:C_0402_1005Metric, F.Cu at (86.6, 77.4)
- added C32: 100nF, Capacitor_SMD:C_0402_1005Metric, F.Cu at (105.7, 77.4)
- added C33: 100nF, Capacitor_SMD:C_0402_1005Metric, F.Cu at (124.7, 77.4)
- added C34: 100nF, Capacitor_SMD:C_0402_1005Metric, F.Cu at (143.8, 77.4)
- added C35: 100nF, Capacitor_SMD:C_0402_1005Metric, F.Cu at (162.8, 77.4)
- added C36: 100nF, Capacitor_SMD:C_0402_1005Metric, F.Cu at (181.9, 77.4)
- added C37: 100nF, Capacitor_SMD:C_0402_1005Metric, F.Cu at (200.9, 77.4)
- added C38: 100nF, Capacitor_SMD:C_0402_1005Metric, F.Cu at (220.0, 77.4)
- added C39: 100nF, Capacitor_SMD:C_0402_1005Metric, F.Cu at (239.0, 77.4)
- added C4: 100nF, Capacitor_SMD:C_0402_1005Metric, F.Cu at (156.5, 34.5)
- added C40: 100nF, Capacitor_SMD:C_0402_1005Metric, F.Cu at (258.1, 77.4)
- added C41: 100nF, Capacitor_SMD:C_0402_1005Metric, F.Cu at (277.1, 77.4)
- added C42: 100nF, Capacitor_SMD:C_0402_1005Metric, F.Cu at (296.2, 77.4)
- added C43: 100nF, Capacitor_SMD:C_0402_1005Metric, F.Cu at (324.7, 77.4)
- added C44: 100nF, Capacitor_SMD:C_0402_1005Metric, F.Cu at (360.0, 77.4)
- added C45: 100nF, Capacitor_SMD:C_0402_1005Metric, F.Cu at (379.0, 77.4)
- added C46: 100nF, Capacitor_SMD:C_0402_1005Metric, F.Cu at (398.1, 77.4)
- added C47: 100nF, Capacitor_SMD:C_0402_1005Metric, F.Cu at (423.8, 77.4)
- added C48: 100nF, Capacitor_SMD:C_0402_1005Metric, F.Cu at (442.8, 77.4)
- added C49: 100nF, Capacitor_SMD:C_0402_1005Metric, F.Cu at (461.9, 77.4)
- added C50: 100nF, Capacitor_SMD:C_0402_1005Metric, F.Cu at (480.9, 77.4)
- added C51: 100nF, Capacitor_SMD:C_0402_1005Metric, F.Cu at (43.6, 96.4)
- added C52: 100nF, Capacitor_SMD:C_0402_1005Metric, F.Cu at (72.3, 96.4)
- added C53: 100nF, Capacitor_SMD:C_0402_1005Metric, F.Cu at (96.1, 96.4)
- added C54: 100nF, Capacitor_SMD:C_0402_1005Metric, F.Cu at (115.2, 96.4)
- added C55: 100nF, Capacitor_SMD:C_0402_1005Metric, F.Cu at (134.2, 96.4)
- added C56: 100nF, Capacitor_SMD:C_0402_1005Metric, F.Cu at (153.3, 96.4)
- added C57: 100nF, Capacitor_SMD:C_0402_1005Metric, F.Cu at (172.3, 96.4)
- added C58: 100nF, Capacitor_SMD:C_0402_1005Metric, F.Cu at (191.4, 96.4)
- added C59: 100nF, Capacitor_SMD:C_0402_1005Metric, F.Cu at (210.4, 96.4)
- added C60: 100nF, Capacitor_SMD:C_0402_1005Metric, F.Cu at (229.5, 96.4)
- added C61: 100nF, Capacitor_SMD:C_0402_1005Metric, F.Cu at (248.5, 96.4)
- added C62: 100nF, Capacitor_SMD:C_0402_1005Metric, F.Cu at (267.6, 96.4)
- added C63: 100nF, Capacitor_SMD:C_0402_1005Metric, F.Cu at (286.6, 96.4)
- added C64: 100nF, Capacitor_SMD:C_0402_1005Metric, F.Cu at (305.7, 96.4)
- added C65: 100nF, Capacitor_SMD:C_0402_1005Metric, F.Cu at (329.5, 96.4)
- added C66: 100nF, Capacitor_SMD:C_0402_1005Metric, F.Cu at (360.0, 96.4)
- added C67: 100nF, Capacitor_SMD:C_0402_1005Metric, F.Cu at (379.0, 96.4)
- added C68: 100nF, Capacitor_SMD:C_0402_1005Metric, F.Cu at (398.1, 96.4)
- added C69: 100nF, Capacitor_SMD:C_0402_1005Metric, F.Cu at (423.8, 96.4)
- added C70: 100nF, Capacitor_SMD:C_0402_1005Metric, F.Cu at (442.8, 96.4)
- added C71: 100nF, Capacitor_SMD:C_0402_1005Metric, F.Cu at (461.9, 96.4)
- added C72: 100nF, Capacitor_SMD:C_0402_1005Metric, F.Cu at (480.9, 105.9)
- added C73: 100nF, Capacitor_SMD:C_0402_1005Metric, F.Cu at (43.6, 115.5)
- added C74: 100nF, Capacitor_SMD:C_0402_1005Metric, F.Cu at (72.3, 115.5)
- added C75: 100nF, Capacitor_SMD:C_0402_1005Metric, F.Cu at (100.9, 115.5)
- added C76: 100nF, Capacitor_SMD:C_0402_1005Metric, F.Cu at (120.0, 115.5)
- added C77: 100nF, Capacitor_SMD:C_0402_1005Metric, F.Cu at (139.0, 115.5)
- added C78: 100nF, Capacitor_SMD:C_0402_1005Metric, F.Cu at (158.1, 115.5)
- added C79: 100nF, Capacitor_SMD:C_0402_1005Metric, F.Cu at (177.1, 115.5)
- added C80: 100nF, Capacitor_SMD:C_0402_1005Metric, F.Cu at (196.2, 115.5)
- added C81: 100nF, Capacitor_SMD:C_0402_1005Metric, F.Cu at (215.2, 115.5)
- added C82: 100nF, Capacitor_SMD:C_0402_1005Metric, F.Cu at (234.3, 115.5)
- added C83: 100nF, Capacitor_SMD:C_0402_1005Metric, F.Cu at (253.3, 115.5)
- added C84: 100nF, Capacitor_SMD:C_0402_1005Metric, F.Cu at (272.4, 115.5)
- added C85: 100nF, Capacitor_SMD:C_0402_1005Metric, F.Cu at (291.4, 115.5)
- added C86: 100nF, Capacitor_SMD:C_0402_1005Metric, F.Cu at (322.4, 115.5)
- added C87: 100nF, Capacitor_SMD:C_0402_1005Metric, F.Cu at (423.8, 115.5)
- added C88: 100nF, Capacitor_SMD:C_0402_1005Metric, F.Cu at (442.8, 115.5)
- added C89: 100nF, Capacitor_SMD:C_0402_1005Metric, F.Cu at (461.9, 115.5)
- added C90: 100nF, Capacitor_SMD:C_0402_1005Metric, F.Cu at (43.6, 134.5)
- added C91: 100nF, Capacitor_SMD:C_0402_1005Metric, F.Cu at (79.5, 134.5)
- added C92: 100nF, Capacitor_SMD:C_0402_1005Metric, F.Cu at (110.4, 134.5)
- added C93: 100nF, Capacitor_SMD:C_0402_1005Metric, F.Cu at (129.5, 134.5)
- added C94: 100nF, Capacitor_SMD:C_0402_1005Metric, F.Cu at (148.5, 134.5)
- added C95: 100nF, Capacitor_SMD:C_0402_1005Metric, F.Cu at (167.6, 134.5)
- added C96: 100nF, Capacitor_SMD:C_0402_1005Metric, F.Cu at (186.6, 134.5)
- added C97: 100nF, Capacitor_SMD:C_0402_1005Metric, F.Cu at (205.7, 134.5)
- added C98: 100nF, Capacitor_SMD:C_0402_1005Metric, F.Cu at (224.7, 134.5)
- added C99: 100nF, Capacitor_SMD:C_0402_1005Metric, F.Cu at (243.8, 134.5)
- added D100: B140S1F-7, Diode_SMD:D_SOD-123F, F.Cu at (252.9, 136.6)
- added D101: B140S1F-7, Diode_SMD:D_SOD-123F, F.Cu at (272.0, 136.6)
- added D102: B140S1F-7, Diode_SMD:D_SOD-123F, F.Cu at (307.7, 136.6)
- added D103: B140S1F-7, Diode_SMD:D_SOD-123F, F.Cu at (369.1, 136.6)
- added D104: B140S1F-7, Diode_SMD:D_SOD-123F, F.Cu at (413.9, 136.6)
- added D105: B140S1F-7, Diode_SMD:D_SOD-123F, F.Cu at (432.9, 136.6)
- added D106: B140S1F-7, Diode_SMD:D_SOD-123F, F.Cu at (452.0, 136.6)
- added D107: B140S1F-7, Diode_SMD:D_SOD-123F, F.Cu at (471.0, 146.1)
- added D108: B140S1F-7, Diode_SMD:D_SOD-123F, F.Cu at (33.7, 155.7)
- added D109: B140S1F-7, Diode_SMD:D_SOD-123F, F.Cu at (62.4, 155.7)
- added D110: B140S1F-7, Diode_SMD:D_SOD-123F, F.Cu at (88.6, 155.7)
- added D111: B140S1F-7, Diode_SMD:D_SOD-123F, F.Cu at (112.4, 155.7)
- added D112: B140S1F-7, Diode_SMD:D_SOD-123F, F.Cu at (179.1, 155.7)
- added D113: B140S1F-7, Diode_SMD:D_SOD-123F, F.Cu at (245.8, 155.7)
- added D114: B140S1F-7, Diode_SMD:D_SOD-123F, F.Cu at (269.6, 155.7)
- added D115: B140S1F-7, Diode_SMD:D_SOD-123F, F.Cu at (293.4, 155.7)
- added D116: B140S1F-7, Diode_SMD:D_SOD-123F, F.Cu at (319.6, 155.7)
- added D117: B140S1F-7, Diode_SMD:D_SOD-123F, F.Cu at (350.1, 155.7)
- added D118: B140S1F-7, Diode_SMD:D_SOD-123F, F.Cu at (369.1, 155.7)
- added D119: B140S1F-7, Diode_SMD:D_SOD-123F, F.Cu at (388.2, 155.7)
- added D120: B140S1F-7, Diode_SMD:D_SOD-123F, F.Cu at (423.4, 155.7)
- added D121: B140S1F-7, Diode_SMD:D_SOD-123F, F.Cu at (452.0, 155.7)
- added D122: LED, keyboard:LED_0603_1608Metric, F.Cu at (-47.5, -27.8)
- added D123: LED, keyboard:LED_0603_1608Metric, F.Cu at (-47.5, -25.3)
- added D66: B140S1F-7, Diode_SMD:D_SOD-123F, F.Cu at (350.1, 98.5)
- added D67: B140S1F-7, Diode_SMD:D_SOD-123F, F.Cu at (369.1, 98.5)
- added D68: B140S1F-7, Diode_SMD:D_SOD-123F, F.Cu at (388.2, 98.5)
- added D69: B140S1F-7, Diode_SMD:D_SOD-123F, F.Cu at (413.9, 98.5)
- added D70: B140S1F-7, Diode_SMD:D_SOD-123F, F.Cu at (432.9, 98.5)
- added D71: B140S1F-7, Diode_SMD:D_SOD-123F, F.Cu at (452.0, 98.5)
- added D72: B140S1F-7, Diode_SMD:D_SOD-123F, F.Cu at (471.0, 108.0)
- added D73: B140S1F-7, Diode_SMD:D_SOD-123F, F.Cu at (33.7, 117.6)
- added D74: B140S1F-7, Diode_SMD:D_SOD-123F, F.Cu at (62.4, 117.6)
- added D75: B140S1F-7, Diode_SMD:D_SOD-123F, F.Cu at (91.0, 117.6)
- added D76: B140S1F-7, Diode_SMD:D_SOD-123F, F.Cu at (110.1, 117.6)
- added D77: B140S1F-7, Diode_SMD:D_SOD-123F, F.Cu at (129.1, 117.6)
- added D78: B140S1F-7, Diode_SMD:D_SOD-123F, F.Cu at (148.2, 117.6)
- added D79: B140S1F-7, Diode_SMD:D_SOD-123F, F.Cu at (167.2, 117.6)
- added D80: B140S1F-7, Diode_SMD:D_SOD-123F, F.Cu at (186.3, 117.6)
- added D81: B140S1F-7, Diode_SMD:D_SOD-123F, F.Cu at (205.3, 117.6)
- added D82: B140S1F-7, Diode_SMD:D_SOD-123F, F.Cu at (224.4, 117.6)
- added D83: B140S1F-7, Diode_SMD:D_SOD-123F, F.Cu at (243.4, 117.6)
- added D84: B140S1F-7, Diode_SMD:D_SOD-123F, F.Cu at (262.5, 117.6)
- added D85: B140S1F-7, Diode_SMD:D_SOD-123F, F.Cu at (281.5, 117.6)
- added D86: B140S1F-7, Diode_SMD:D_SOD-123F, F.Cu at (312.5, 117.6)
- added D87: B140S1F-7, Diode_SMD:D_SOD-123F, F.Cu at (413.9, 117.6)
- added D88: B140S1F-7, Diode_SMD:D_SOD-123F, F.Cu at (432.9, 117.6)
- added D89: B140S1F-7, Diode_SMD:D_SOD-123F, F.Cu at (452.0, 117.6)
- added D90: B140S1F-7, Diode_SMD:D_SOD-123F, F.Cu at (33.7, 136.6)
- added D91: B140S1F-7, Diode_SMD:D_SOD-123F, F.Cu at (69.6, 136.6)
- added D92: B140S1F-7, Diode_SMD:D_SOD-123F, F.Cu at (100.5, 136.6)
- added D93: B140S1F-7, Diode_SMD:D_SOD-123F, F.Cu at (119.6, 136.6)
- added D94: B140S1F-7, Diode_SMD:D_SOD-123F, F.Cu at (138.6, 136.6)
- added D95: B140S1F-7, Diode_SMD:D_SOD-123F, F.Cu at (157.7, 136.6)
- added D96: B140S1F-7, Diode_SMD:D_SOD-123F, F.Cu at (176.7, 136.6)
- added D97: B140S1F-7, Diode_SMD:D_SOD-123F, F.Cu at (195.8, 136.6)
- added D98: B140S1F-7, Diode_SMD:D_SOD-123F, F.Cu at (214.8, 136.6)
- added D99: B140S1F-7, Diode_SMD:D_SOD-123F, F.Cu at (233.9, 136.6)
- added J2: Tag connect TC2030-CTX, keyboard:TC2030-IDC-NL, F.Cu at (-32.9, 15.5)
- added LED1: WS2812B, LED_SMD:LED_WS2812B_PLCC4_5.0x5.0mm_P3.2mm, F.Cu at (94.5, 32.9)
- added LED10: WS2812B, LED_SMD:LED_WS2812B_PLCC4_5.0x5.0mm_P3.2mm, F.Cu at (94.5, 52.0)
- added LED100: WS2812B, LED_SMD:LED_WS2812B_PLCC4_5.0x5.0mm_P3.2mm, F.Cu at (258.0, 132.9)
- added LED101: WS2812B, LED_SMD:LED_WS2812B_PLCC4_5.0x5.0mm_P3.2mm, F.Cu at (277.1, 132.9)
- added LED102: WS2812B, LED_SMD:LED_WS2812B_PLCC4_5.0x5.0mm_P3.2mm, F.Cu at (312.8, 132.9)
- added LED103: WS2812B, LED_SMD:LED_WS2812B_PLCC4_5.0x5.0mm_P3.2mm, F.Cu at (374.2, 132.9)
- added LED104: WS2812B, LED_SMD:LED_WS2812B_PLCC4_5.0x5.0mm_P3.2mm, F.Cu at (419.0, 132.9)
- added LED105: WS2812B, LED_SMD:LED_WS2812B_PLCC4_5.0x5.0mm_P3.2mm, F.Cu at (438.0, 132.9)
- added LED106: WS2812B, LED_SMD:LED_WS2812B_PLCC4_5.0x5.0mm_P3.2mm, F.Cu at (457.1, 132.9)
- added LED107: WS2812B, LED_SMD:LED_WS2812B_PLCC4_5.0x5.0mm_P3.2mm, F.Cu at (476.1, 142.4)
- added LED108: WS2812B, LED_SMD:LED_WS2812B_PLCC4_5.0x5.0mm_P3.2mm, F.Cu at (38.8, 152.0)
- added LED109: WS2812B, LED_SMD:LED_WS2812B_PLCC4_5.0x5.0mm_P3.2mm, F.Cu at (67.5, 152.0)
- added LED11: WS2812B, LED_SMD:LED_WS2812B_PLCC4_5.0x5.0mm_P3.2mm, F.Cu at (113.6, 52.0)
- added LED110: WS2812B, LED_SMD:LED_WS2812B_PLCC4_5.0x5.0mm_P3.2mm, F.Cu at (93.7, 152.0)
- added LED111: WS2812B, LED_SMD:LED_WS2812B_PLCC4_5.0x5.0mm_P3.2mm, F.Cu at (117.5, 152.0)
- added LED112: WS2812B, LED_SMD:LED_WS2812B_PLCC4_5.0x5.0mm_P3.2mm, F.Cu at (184.2, 152.0)
- added LED113: WS2812B, LED_SMD:LED_WS2812B_PLCC4_5.0x5.0mm_P3.2mm, F.Cu at (250.9, 152.0)
- added LED114: WS2812B, LED_SMD:LED_WS2812B_PLCC4_5.0x5.0mm_P3.2mm, F.Cu at (274.7, 152.0)
- added LED115: WS2812B, LED_SMD:LED_WS2812B_PLCC4_5.0x5.0mm_P3.2mm, F.Cu at (298.5, 152.0)
- added LED116: WS2812B, LED_SMD:LED_WS2812B_PLCC4_5.0x5.0mm_P3.2mm, F.Cu at (324.7, 152.0)
- added LED117: WS2812B, LED_SMD:LED_WS2812B_PLCC4_5.0x5.0mm_P3.2mm, F.Cu at (355.2, 152.0)
- added LED118: WS2812B, LED_SMD:LED_WS2812B_PLCC4_5.0x5.0mm_P3.2mm, F.Cu at (374.2, 152.0)
- added LED119: WS2812B, LED_SMD:LED_WS2812B_PLCC4_5.0x5.0mm_P3.2mm, F.Cu at (393.3, 152.0)
- added LED12: WS2812B, LED_SMD:LED_WS2812B_PLCC4_5.0x5.0mm_P3.2mm, F.Cu at (132.6, 52.0)
- added LED120: WS2812B, LED_SMD:LED_WS2812B_PLCC4_5.0x5.0mm_P3.2mm, F.Cu at (428.5, 152.0)
- added LED121: WS2812B, LED_SMD:LED_WS2812B_PLCC4_5.0x5.0mm_P3.2mm, F.Cu at (457.1, 152.0)
- added LED13: WS2812B, LED_SMD:LED_WS2812B_PLCC4_5.0x5.0mm_P3.2mm, F.Cu at (151.7, 52.0)
- added LED14: WS2812B, LED_SMD:LED_WS2812B_PLCC4_5.0x5.0mm_P3.2mm, F.Cu at (183.4, 52.0)
- added LED15: WS2812B, LED_SMD:LED_WS2812B_PLCC4_5.0x5.0mm_P3.2mm, F.Cu at (202.5, 52.0)
- added LED16: WS2812B, LED_SMD:LED_WS2812B_PLCC4_5.0x5.0mm_P3.2mm, F.Cu at (221.5, 52.0)
- added LED17: WS2812B, LED_SMD:LED_WS2812B_PLCC4_5.0x5.0mm_P3.2mm, F.Cu at (240.6, 52.0)
- added LED18: WS2812B, LED_SMD:LED_WS2812B_PLCC4_5.0x5.0mm_P3.2mm, F.Cu at (272.3, 52.0)
- added LED19: WS2812B, LED_SMD:LED_WS2812B_PLCC4_5.0x5.0mm_P3.2mm, F.Cu at (291.4, 52.0)
- added LED2: WS2812B, LED_SMD:LED_WS2812B_PLCC4_5.0x5.0mm_P3.2mm, F.Cu at (113.6, 32.9)
- added LED20: WS2812B, LED_SMD:LED_WS2812B_PLCC4_5.0x5.0mm_P3.2mm, F.Cu at (310.4, 52.0)
- added LED21: WS2812B, LED_SMD:LED_WS2812B_PLCC4_5.0x5.0mm_P3.2mm, F.Cu at (329.5, 52.0)
- added LED22: WS2812B, LED_SMD:LED_WS2812B_PLCC4_5.0x5.0mm_P3.2mm, F.Cu at (355.2, 52.0)
- added LED23: WS2812B, LED_SMD:LED_WS2812B_PLCC4_5.0x5.0mm_P3.2mm, F.Cu at (374.2, 52.0)
- added LED24: WS2812B, LED_SMD:LED_WS2812B_PLCC4_5.0x5.0mm_P3.2mm, F.Cu at (393.3, 52.0)
- added LED25: WS2812B, LED_SMD:LED_WS2812B_PLCC4_5.0x5.0mm_P3.2mm, F.Cu at (419.0, 52.0)
- added LED26: WS2812B, LED_SMD:LED_WS2812B_PLCC4_5.0x5.0mm_P3.2mm, F.Cu at (438.1, 52.0)
- added LED27: WS2812B, LED_SMD:LED_WS2812B_PLCC4_5.0x5.0mm_P3.2mm, F.Cu at (457.1, 52.0)
- added LED28: WS2812B, LED_SMD:LED_WS2812B_PLCC4_5.0x5.0mm_P3.2mm, F.Cu at (476.2, 52.0)
- added LED29: WS2812B, LED_SMD:LED_WS2812B_PLCC4_5.0x5.0mm_P3.2mm, F.Cu at (38.8, 75.8)
- added LED3: WS2812B, LED_SMD:LED_WS2812B_PLCC4_5.0x5.0mm_P3.2mm, F.Cu at (132.6, 32.9)
- added LED30: WS2812B, LED_SMD:LED_WS2812B_PLCC4_5.0x5.0mm_P3.2mm, F.Cu at (62.8, 75.8)
- added LED31: WS2812B, LED_SMD:LED_WS2812B_PLCC4_5.0x5.0mm_P3.2mm, F.Cu at (81.8, 75.8)
- added LED32: WS2812B, LED_SMD:LED_WS2812B_PLCC4_5.0x5.0mm_P3.2mm, F.Cu at (100.9, 75.8)
- added LED33: WS2812B, LED_SMD:LED_WS2812B_PLCC4_5.0x5.0mm_P3.2mm, F.Cu at (119.9, 75.8)
- added LED34: WS2812B, LED_SMD:LED_WS2812B_PLCC4_5.0x5.0mm_P3.2mm, F.Cu at (139.0, 75.8)
- added LED35: WS2812B, LED_SMD:LED_WS2812B_PLCC4_5.0x5.0mm_P3.2mm, F.Cu at (158.0, 75.8)
- added LED36: WS2812B, LED_SMD:LED_WS2812B_PLCC4_5.0x5.0mm_P3.2mm, F.Cu at (177.1, 75.8)
- added LED37: WS2812B, LED_SMD:LED_WS2812B_PLCC4_5.0x5.0mm_P3.2mm, F.Cu at (196.1, 75.8)
- added LED38: WS2812B, LED_SMD:LED_WS2812B_PLCC4_5.0x5.0mm_P3.2mm, F.Cu at (215.2, 75.8)
- added LED39: WS2812B, LED_SMD:LED_WS2812B_PLCC4_5.0x5.0mm_P3.2mm, F.Cu at (234.2, 75.8)
- added LED4: WS2812B, LED_SMD:LED_WS2812B_PLCC4_5.0x5.0mm_P3.2mm, F.Cu at (151.7, 32.9)
- added LED40: WS2812B, LED_SMD:LED_WS2812B_PLCC4_5.0x5.0mm_P3.2mm, F.Cu at (253.3, 75.8)
- added LED41: WS2812B, LED_SMD:LED_WS2812B_PLCC4_5.0x5.0mm_P3.2mm, F.Cu at (272.3, 75.8)
- added LED42: WS2812B, LED_SMD:LED_WS2812B_PLCC4_5.0x5.0mm_P3.2mm, F.Cu at (291.4, 75.8)
- added LED43: WS2812B, LED_SMD:LED_WS2812B_PLCC4_5.0x5.0mm_P3.2mm, F.Cu at (319.9, 75.8)
- added LED44: WS2812B, LED_SMD:LED_WS2812B_PLCC4_5.0x5.0mm_P3.2mm, F.Cu at (355.2, 75.8)
- added LED45: WS2812B, LED_SMD:LED_WS2812B_PLCC4_5.0x5.0mm_P3.2mm, F.Cu at (374.2, 75.8)
- added LED46: WS2812B, LED_SMD:LED_WS2812B_PLCC4_5.0x5.0mm_P3.2mm, F.Cu at (393.3, 75.8)
- added LED47: WS2812B, LED_SMD:LED_WS2812B_PLCC4_5.0x5.0mm_P3.2mm, F.Cu at (419.0, 75.8)
- added LED48: WS2812B, LED_SMD:LED_WS2812B_PLCC4_5.0x5.0mm_P3.2mm, F.Cu at (438.0, 75.8)
- added LED49: WS2812B, LED_SMD:LED_WS2812B_PLCC4_5.0x5.0mm_P3.2mm, F.Cu at (457.1, 75.8)
- added LED5: WS2812B, LED_SMD:LED_WS2812B_PLCC4_5.0x5.0mm_P3.2mm, F.Cu at (183.4, 32.9)
- added LED50: WS2812B, LED_SMD:LED_WS2812B_PLCC4_5.0x5.0mm_P3.2mm, F.Cu at (476.1, 75.8)
- added LED51: WS2812B, LED_SMD:LED_WS2812B_PLCC4_5.0x5.0mm_P3.2mm, F.Cu at (38.8, 94.8)
- added LED52: WS2812B, LED_SMD:LED_WS2812B_PLCC4_5.0x5.0mm_P3.2mm, F.Cu at (67.5, 94.8)
- added LED53: WS2812B, LED_SMD:LED_WS2812B_PLCC4_5.0x5.0mm_P3.2mm, F.Cu at (91.3, 94.8)
- added LED54: WS2812B, LED_SMD:LED_WS2812B_PLCC4_5.0x5.0mm_P3.2mm, F.Cu at (110.4, 94.8)
- added LED55: WS2812B, LED_SMD:LED_WS2812B_PLCC4_5.0x5.0mm_P3.2mm, F.Cu at (129.4, 94.8)
- added LED56: WS2812B, LED_SMD:LED_WS2812B_PLCC4_5.0x5.0mm_P3.2mm, F.Cu at (148.5, 94.8)
- added LED57: WS2812B, LED_SMD:LED_WS2812B_PLCC4_5.0x5.0mm_P3.2mm, F.Cu at (167.5, 94.8)
- added LED58: WS2812B, LED_SMD:LED_WS2812B_PLCC4_5.0x5.0mm_P3.2mm, F.Cu at (186.6, 94.8)
- added LED59: WS2812B, LED_SMD:LED_WS2812B_PLCC4_5.0x5.0mm_P3.2mm, F.Cu at (205.6, 94.8)
- added LED6: WS2812B, LED_SMD:LED_WS2812B_PLCC4_5.0x5.0mm_P3.2mm, F.Cu at (202.5, 32.9)
- added LED60: WS2812B, LED_SMD:LED_WS2812B_PLCC4_5.0x5.0mm_P3.2mm, F.Cu at (224.7, 94.8)
- added LED61: WS2812B, LED_SMD:LED_WS2812B_PLCC4_5.0x5.0mm_P3.2mm, F.Cu at (243.7, 94.8)
- added LED62: WS2812B, LED_SMD:LED_WS2812B_PLCC4_5.0x5.0mm_P3.2mm, F.Cu at (262.8, 94.8)
- added LED63: WS2812B, LED_SMD:LED_WS2812B_PLCC4_5.0x5.0mm_P3.2mm, F.Cu at (281.8, 94.8)
- added LED64: WS2812B, LED_SMD:LED_WS2812B_PLCC4_5.0x5.0mm_P3.2mm, F.Cu at (300.9, 94.8)
- added LED65: WS2812B, LED_SMD:LED_WS2812B_PLCC4_5.0x5.0mm_P3.2mm, F.Cu at (324.7, 94.8)
- added LED66: WS2812B, LED_SMD:LED_WS2812B_PLCC4_5.0x5.0mm_P3.2mm, F.Cu at (355.2, 94.8)
- added LED67: WS2812B, LED_SMD:LED_WS2812B_PLCC4_5.0x5.0mm_P3.2mm, F.Cu at (374.2, 94.8)
- added LED68: WS2812B, LED_SMD:LED_WS2812B_PLCC4_5.0x5.0mm_P3.2mm, F.Cu at (393.3, 94.8)
- added LED69: WS2812B, LED_SMD:LED_WS2812B_PLCC4_5.0x5.0mm_P3.2mm, F.Cu at (419.0, 94.8)
- added LED7: WS2812B, LED_SMD:LED_WS2812B_PLCC4_5.0x5.0mm_P3.2mm, F.Cu at (221.5, 32.9)
- added LED70: WS2812B, LED_SMD:LED_WS2812B_PLCC4_5.0x5.0mm_P3.2mm, F.Cu at (438.0, 94.8)
- added LED71: WS2812B, LED_SMD:LED_WS2812B_PLCC4_5.0x5.0mm_P3.2mm, F.Cu at (457.1, 94.8)
- added LED72: WS2812B, LED_SMD:LED_WS2812B_PLCC4_5.0x5.0mm_P3.2mm, F.Cu at (476.1, 104.3)
- added LED73: WS2812B, LED_SMD:LED_WS2812B_PLCC4_5.0x5.0mm_P3.2mm, F.Cu at (38.8, 113.9)
- added LED74: WS2812B, LED_SMD:LED_WS2812B_PLCC4_5.0x5.0mm_P3.2mm, F.Cu at (67.5, 113.9)
- added LED75: WS2812B, LED_SMD:LED_WS2812B_PLCC4_5.0x5.0mm_P3.2mm, F.Cu at (96.1, 113.9)
- added LED76: WS2812B, LED_SMD:LED_WS2812B_PLCC4_5.0x5.0mm_P3.2mm, F.Cu at (115.2, 113.9)
- added LED77: WS2812B, LED_SMD:LED_WS2812B_PLCC4_5.0x5.0mm_P3.2mm, F.Cu at (134.2, 113.9)
- added LED78: WS2812B, LED_SMD:LED_WS2812B_PLCC4_5.0x5.0mm_P3.2mm, F.Cu at (153.3, 113.9)
- added LED79: WS2812B, LED_SMD:LED_WS2812B_PLCC4_5.0x5.0mm_P3.2mm, F.Cu at (172.3, 113.9)
- added LED8: WS2812B, LED_SMD:LED_WS2812B_PLCC4_5.0x5.0mm_P3.2mm, F.Cu at (240.6, 32.9)
- added LED80: WS2812B, LED_SMD:LED_WS2812B_PLCC4_5.0x5.0mm_P3.2mm, F.Cu at (191.4, 113.9)
- added LED81: WS2812B, LED_SMD:LED_WS2812B_PLCC4_5.0x5.0mm_P3.2mm, F.Cu at (210.4, 113.9)
- added LED82: WS2812B, LED_SMD:LED_WS2812B_PLCC4_5.0x5.0mm_P3.2mm, F.Cu at (229.5, 113.9)
- added LED83: WS2812B, LED_SMD:LED_WS2812B_PLCC4_5.0x5.0mm_P3.2mm, F.Cu at (248.5, 113.9)
- added LED84: WS2812B, LED_SMD:LED_WS2812B_PLCC4_5.0x5.0mm_P3.2mm, F.Cu at (267.6, 113.9)
- added LED85: WS2812B, LED_SMD:LED_WS2812B_PLCC4_5.0x5.0mm_P3.2mm, F.Cu at (286.6, 113.9)
- added LED86: WS2812B, LED_SMD:LED_WS2812B_PLCC4_5.0x5.0mm_P3.2mm, F.Cu at (317.6, 113.9)
- added LED87: WS2812B, LED_SMD:LED_WS2812B_PLCC4_5.0x5.0mm_P3.2mm, F.Cu at (419.0, 113.9)
- added LED88: WS2812B, LED_SMD:LED_WS2812B_PLCC4_5.0x5.0mm_P3.2mm, F.Cu at (438.0, 113.9)
- added LED89: WS2812B, LED_SMD:LED_WS2812B_PLCC4_5.0x5.0mm_P3.2mm, F.Cu at (457.1, 113.9)
- added LED9: WS2812B, LED_SMD:LED_WS2812B_PLCC4_5.0x5.0mm_P3.2mm, F.Cu at (62.8, 52.0)
- added LED90: WS2812B, LED_SMD:LED_WS2812B_PLCC4_5.0x5.0mm_P3.2mm, F.Cu at (38.8, 132.9)
- added LED91: WS2812B, LED_SMD:LED_WS2812B_PLCC4_5.0x5.0mm_P3.2mm, F.Cu at (74.7, 132.9)
- added LED92: WS2812B, LED_SMD:LED_WS2812B_PLCC4_5.0x5.0mm_P3.2mm, F.Cu at (105.6, 132.9)
- added LED93: WS2812B, LED_SMD:LED_WS2812B_PLCC4_5.0x5.0mm_P3.2mm, F.Cu at (124.7, 132.9)
- added LED94: WS2812B, LED_SMD:LED_WS2812B_PLCC4_5.0x5.0mm_P3.2mm, F.Cu at (143.7, 132.9)
- added LED95: WS2812B, LED_SMD:LED_WS2812B_PLCC4_5.0x5.0mm_P3.2mm, F.Cu at (162.8, 132.9)
- added LED96: WS2812B, LED_SMD:LED_WS2812B_PLCC4_5.0x5.0mm_P3.2mm, F.Cu at (181.8, 132.9)
- added LED97: WS2812B, LED_SMD:LED_WS2812B_PLCC4_5.0x5.0mm_P3.2mm, F.Cu at (200.9, 132.9)
- added LED98: WS2812B, LED_SMD:LED_WS2812B_PLCC4_5.0x5.0mm_P3.2mm, F.Cu at (219.9, 132.9)
- added LED99: WS2812B, LED_SMD:LED_WS2812B_PLCC4_5.0x5.0mm_P3.2mm, F.Cu at (239.0, 132.9)
- added MX100: 1.00u, key-switches:SW_Gateron_LowProfile_HotSwap_PTH, F.Cu at (258.8, 138.1)
- added MX101: 1.00u, key-switches:SW_Gateron_LowProfile_HotSwap_PTH, F.Cu at (277.8, 138.1)
- added MX102: 1.00u, key-switches:SW_Gateron_LowProfile_HotSwap_PTH, F.Cu at (313.5, 138.1)
- added MX103: 1.00u, key-switches:SW_Gateron_LowProfile_HotSwap_PTH, F.Cu at (375.0, 138.1)
- added MX104: 1.00u, key-switches:SW_Gateron_LowProfile_HotSwap_PTH, F.Cu at (419.7, 138.1)
- added MX105: 1.00u, key-switches:SW_Gateron_LowProfile_HotSwap_PTH, F.Cu at (438.8, 138.1)
- added MX106: 1.00u, key-switches:SW_Gateron_LowProfile_HotSwap_PTH, F.Cu at (457.8, 138.1)
- added MX107: 1.00u, key-switches:SW_Gateron_LowProfile_HotSwap_PTH, F.Cu at (476.9, 147.6)
- added MX108: 1.00u, key-switches:SW_Gateron_LowProfile_HotSwap_PTH, F.Cu at (39.5, 157.2)
- added MX109: 1.00u, key-switches:SW_Gateron_LowProfile_HotSwap_PTH, F.Cu at (68.3, 157.2)
- added MX110: 1.00u, key-switches:SW_Gateron_LowProfile_HotSwap_PTH, F.Cu at (94.5, 157.2)
- added MX111: 1.00u, key-switches:SW_Gateron_LowProfile_HotSwap_PTH, F.Cu at (118.3, 157.2)
- added MX112: 1.00u, key-switches:SW_Gateron_LowProfile_HotSwap_PTH, F.Cu at (184.9, 157.2)
- added MX113: 1.00u, key-switches:SW_Gateron_LowProfile_HotSwap_PTH, F.Cu at (251.6, 157.2)
- added MX114: 1.00u, key-switches:SW_Gateron_LowProfile_HotSwap_PTH, F.Cu at (275.4, 157.2)
- added MX115: 1.00u, key-switches:SW_Gateron_LowProfile_HotSwap_PTH, F.Cu at (299.2, 157.2)
- added MX116: 1.00u, key-switches:SW_Gateron_LowProfile_HotSwap_PTH, F.Cu at (325.4, 157.2)
- added MX117: 1.00u, key-switches:SW_Gateron_LowProfile_HotSwap_PTH, F.Cu at (355.9, 157.2)
- added MX118: 1.00u, key-switches:SW_Gateron_LowProfile_HotSwap_PTH, F.Cu at (375.0, 157.2)
- added MX119: 1.00u, key-switches:SW_Gateron_LowProfile_HotSwap_PTH, F.Cu at (394.0, 157.2)
- added MX120: 1.00u, key-switches:SW_Gateron_LowProfile_HotSwap_PTH, F.Cu at (429.3, 157.2)
- added MX121: 1.00u, key-switches:SW_Gateron_LowProfile_HotSwap_PTH, F.Cu at (457.8, 157.2)
- added MX74: 1.00u, key-switches:SW_Gateron_LowProfile_HotSwap_PTH, F.Cu at (68.3, 119.1)
- added MX75: 1.00u, key-switches:SW_Gateron_LowProfile_HotSwap_PTH, F.Cu at (96.8, 119.1)
- added MX76: 1.00u, key-switches:SW_Gateron_LowProfile_HotSwap_PTH, F.Cu at (115.9, 119.1)
- added MX77: 1.00u, key-switches:SW_Gateron_LowProfile_HotSwap_PTH, F.Cu at (134.9, 119.1)
- added MX78: 1.00u, key-switches:SW_Gateron_LowProfile_HotSwap_PTH, F.Cu at (154.0, 119.1)
- added MX79: 1.00u, key-switches:SW_Gateron_LowProfile_HotSwap_PTH, F.Cu at (173.0, 119.1)
- added MX80: 1.00u, key-switches:SW_Gateron_LowProfile_HotSwap_PTH, F.Cu at (192.1, 119.1)
- added MX81: 1.00u, key-switches:SW_Gateron_LowProfile_HotSwap_PTH, F.Cu at (211.1, 119.1)
- added MX82: 1.00u, key-switches:SW_Gateron_LowProfile_HotSwap_PTH, F.Cu at (230.2, 119.1)
- added MX83: 1.00u, key-switches:SW_Gateron_LowProfile_HotSwap_PTH, F.Cu at (249.2, 119.1)
- added MX84: 1.00u, key-switches:SW_Gateron_LowProfile_HotSwap_PTH, F.Cu at (268.3, 119.1)
- added MX85: 1.00u, key-switches:SW_Gateron_LowProfile_HotSwap_PTH, F.Cu at (287.3, 119.1)
- added MX86: 1.00u, key-switches:SW_Gateron_LowProfile_HotSwap_PTH, F.Cu at (318.3, 119.1)
- added MX87: 1.00u, key-switches:SW_Gateron_LowProfile_HotSwap_PTH, F.Cu at (419.7, 119.1)
- added MX88: 1.00u, key-switches:SW_Gateron_LowProfile_HotSwap_PTH, F.Cu at (438.8, 119.1)
- added MX89: 1.00u, key-switches:SW_Gateron_LowProfile_HotSwap_PTH, F.Cu at (457.8, 119.1)
- added MX90: 1.00u, key-switches:SW_Gateron_LowProfile_HotSwap_PTH, F.Cu at (39.5, 138.1)
- added MX91: 1.00u, key-switches:SW_Gateron_LowProfile_HotSwap_PTH, F.Cu at (75.4, 138.1)
- added MX92: 1.00u, key-switches:SW_Gateron_LowProfile_HotSwap_PTH, F.Cu at (106.4, 138.1)
- added MX93: 1.00u, key-switches:SW_Gateron_LowProfile_HotSwap_PTH, F.Cu at (125.4, 138.1)
- added MX94: 1.00u, key-switches:SW_Gateron_LowProfile_HotSwap_PTH, F.Cu at (144.5, 138.1)
- added MX95: 1.00u, key-switches:SW_Gateron_LowProfile_HotSwap_PTH, F.Cu at (163.5, 138.1)
- added MX96: 1.00u, key-switches:SW_Gateron_LowProfile_HotSwap_PTH, F.Cu at (182.6, 138.1)
- added MX97: 1.00u, key-switches:SW_Gateron_LowProfile_HotSwap_PTH, F.Cu at (201.6, 138.1)
- added MX98: 1.00u, key-switches:SW_Gateron_LowProfile_HotSwap_PTH, F.Cu at (220.7, 138.1)
- added MX99: 1.00u, key-switches:SW_Gateron_LowProfile_HotSwap_PTH, F.Cu at (239.7, 138.1)
- added R6: 10k, keyboard:R_0402_1005Metric, F.Cu at (-20.0, 18.0)
- added R7: 10k, keyboard:R_0402_1005Metric, F.Cu at (-67.0, -64.9)
- added SW1: Reset Switch, keyboard:RST_SW, F.Cu at (82.3, 302.7)
- added TP1: TestPoint, TestPoint:TestPoint_Pad_D1.5mm, F.Cu at (-19.7, 15.2)
- added U2: SN74AHCT1G125, Package_TO_SOT_SMD:SOT-23-5, F.Cu at (-71.1, -63.5)
- C1, C14, C23: value 1uF -> 100nF; footprint keyboard:C_0603_1608Metric -> Capacitor_SMD:C_0402_1005Metric; moved to F.Cu
- C10: value 1pF -> 100nF; footprint keyboard:C_0402_1005Metric -> Capacitor_SMD:C_0402_1005Metric; moved to F.Cu
- C11: value 1.2pF -> 100nF; footprint keyboard:C_0402_1005Metric -> Capacitor_SMD:C_0402_1005Metric; moved to F.Cu
- C12: value DNP -> 100nF; footprint keyboard:C_0402_1005Metric -> Capacitor_SMD:C_0402_1005Metric; moved to F.Cu
- C13: value 100pF -> 100nF; footprint keyboard:C_0402_1005Metric -> Capacitor_SMD:C_0402_1005Metric; moved to F.Cu
- C16, C17, C24, C25, C26, C27: footprint keyboard:C_0402_1005Metric -> Capacitor_SMD:C_0402_1005Metric; moved to F.Cu
- C2, C20, C21, C22: value 4u7F -> 100nF; footprint keyboard:C_0805_2012Metric -> Capacitor_SMD:C_0402_1005Metric; moved to F.Cu
- C5, C6, C7, C8: value 8pF -> 100nF; footprint keyboard:C_0402_1005Metric -> Capacitor_SMD:C_0402_1005Metric; moved to F.Cu
- C9: value 820pF -> 100nF; footprint keyboard:C_0402_1005Metric -> Capacitor_SMD:C_0402_1005Metric; moved to F.Cu
- D1, D2: value LED -> B140S1F-7; footprint keyboard:LED_0603_1608Metric -> Diode_SMD:D_SOD-123F
- D10, D11, D12, D13, D14, D15, D16, D17, D18, D19, D20, D21, D22, D23, D24, D25, D26, D27, D28, D29, D3, D30, D31, D32, D33, D34, D35, D36, D37, D38, D39, D4, D40, D41, D42, D43, D44, D45, D46, D47, D48, D49, D5, D50, D51, D52, D53, D54, D55, D56, D57, D58, D59, D6, D60, D61, D62, D63, D64, D65, D7, D8, D9: value 1N4148W -> B140S1F-7; footprint keyboard:D_SOD-123 -> Diode_SMD:D_SOD-123F; moved to F.Cu
- J1: value JST-4-pin -> Prog_conn; footprint keyboard:JST-4-pin -> keyboard:DB_CONN
- J3: value Prog_conn -> 53047-0460; footprint keyboard:DB_CONN -> Connector_Molex:Molex_PicoBlade_53048-0410_1x04_P1.25mm_Horizontal
- J5: value Tag connect TC2030-CTX -> JST-4-pin; footprint keyboard:TC2030-IDC-NL -> keyboard:JST-4-pin
- L1: value 4.7nH -> 15nH
- L2: value 60R@100MHz -> 10uH
- L4: value 15nH -> 4.7nH
- L5: value 10uH -> 2.2nH; footprint keyboard:L_0603_1608Metric -> keyboard:L_0402_1005Metric
- L6: value 2.2nH -> 60R@100MHz; footprint keyboard:L_0402_1005Metric -> keyboard:L_0603_1608Metric
- MX1, MX10, MX11, MX12, MX13, MX14, MX15, MX18, MX19, MX2, MX20, MX21, MX22, MX23, MX24, MX25, MX26, MX27, MX28, MX29, MX3, MX33, MX34, MX35, MX36, MX37, MX38, MX39, MX4, MX40, MX41, MX42, MX43, MX46, MX47, MX48, MX49, MX5, MX50, MX51, MX52, MX53, MX54, MX55, MX57, MX6, MX68, MX7, MX72, MX8, MX9: value 1u -> 1.00u; footprint keyboard:SW_Cherry_MX_1.00u_PCB -> key-switches:SW_Gateron_LowProfile_HotSwap_PTH
- MX16: value 2u -> 1.00u; footprint keyboard:SW_Cherry_MX_2.00u_PCB -> key-switches:SW_Gateron_LowProfile_HotSwap_PTH
- MX17, MX30, MX67, MX69, MX71, MX73: value 1.5u -> 1.00u; footprint keyboard:SW_Cherry_MX_1.50u_PCB -> key-switches:SW_Gateron_LowProfile_HotSwap_PTH
- MX31, MX56: value 1.75u -> 1.00u; footprint keyboard:SW_Cherry_MX_1.75u_PCB -> key-switches:SW_Gateron_LowProfile_HotSwap_PTH
- MX32, MX59, MX60, MX61, MX63, MX64, MX65, MX66: value 1.25u -> 1.00u; footprint keyboard:SW_Cherry_MX_1.25u_PCB -> key-switches:SW_Gateron_LowProfile_HotSwap_PTH
- MX44, MX45: value 2.25u -> 1.00u; footprint keyboard:SW_Cherry_MX_2.25u_PCB -> key-switches:SW_Gateron_LowProfile_HotSwap_PTH
- MX58: value 2.75u -> 1.00u; footprint keyboard:SW_Cherry_MX_2.75u_PCB -> key-switches:SW_Gateron_LowProfile_HotSwap_PTH
- MX62: value 6.25u -> 1.00u; footprint keyboard:SW_Cherry_MX_6.25u_PCB -> key-switches:SW_Gateron_LowProfile_HotSwap_PTH
- MX70: value 7u -> 1.00u; footprint keyboard:SW_Cherry_MX_7.00u_PCB -> key-switches:SW_Gateron_LowProfile_HotSwap_PTH
- R1, R2: value 1k2 -> 22E
- R10: value 22E -> 5k1
- R11: value 22E -> 1k2
- R12: value 22E -> 8k2
- R13, R9: value 10k -> 5k1
- R14, R15: value 10k -> 1k2
- R16, R17, R5: value 5k1 -> 10k
- R3: value 8k2 -> 22E
- R4: value 1k2 -> 10k
- R8: value 10k -> 100; footprint keyboard:R_0402_1005Metric -> Resistor_SMD:R_0402_1005Metric
- S2: footprint keyboard:Keybaord_outline_edgecuts -> keyboard:BLE-symbol
- S3: footprint keyboard:BLE-symbol -> keyboard:ZMK_logo
- U1: value BQ24074RGTR -> nRF52840-QIAA-R/nRF52833-QIAA-R; footprint keyboard:QFN-16 -> keyboard:aqfn73
- U3: value nRF52840-QIAA-R/nRF52833-QIAA-R -> TPD4E05U06DQAR; footprint keyboard:aqfn73 -> keyboard:USON-10
- U4: value TPD4E05U06DQAR -> BQ24074RGTR; footprint keyboard:USON-10 -> keyboard:QFN-16
- Y1: value 32MHz -> 32.768kHz; footprint keyboard:SMD-4_crystal -> keyboard:SMD-2_crystal
- Y2: value 32.768kHz -> 32MHz; footprint keyboard:SMD-2_crystal -> keyboard:SMD-4_crystal
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Connections:
- C1 pad 1: /VBUS -> +5V
- C10 pad 1: Net-(U3-ANT) -> +5V
- C11 pad 1: Net-(C11-Pad1) -> +5V
- C12 pad 1: GND -> +5V
- C12 pad 2: Net-(U3-DEC2) -> GND
- C13 pad 1: GND -> +5V
- C13 pad 2: Net-(U3-DEC3) -> GND
- C14 pad 1: Net-(U3-DEC4) -> +5V
- C16 pad 1: /VBATT_nRF -> +5V
- C17 pad 1: GND -> +5V
- C17 pad 2: Net-(U3-DEC4) -> GND
- C2 pad 1: /USB and Power management/V_BATT -> +5V
- C20 pad 1: /VBUS -> +5V
- C21 pad 1: Net-(U3-DECUSB) -> +5V
- C22 pad 1: /VDD_nRF -> +5V
- C23 pad 1: GND -> +5V
- C23 pad 2: /VDD_nRF -> GND
- C24 pad 1: /VDD_nRF -> +5V
- C25 pad 1: /VDD_nRF -> +5V
- C26 pad 1: /VDD_nRF -> +5V
- C27 pad 1: GND -> +5V
- C27 pad 2: Net-(U3-DEC1) -> GND
- C5 pad 1: GND -> +5V
- C5 pad 2: Net-(U3-XC2) -> GND
- C6 pad 1: GND -> +5V
- C6 pad 2: Net-(U3-XC1) -> GND
- C7 pad 1: GND -> +5V
- C7 pad 2: Net-(U3-P0.00/XL1) -> GND
- C8 pad 1: GND -> +5V
- C8 pad 2: Net-(U3-P0.01/XL2) -> GND
- C9 pad 1: GND -> +5V
- C9 pad 2: Net-(U3-DEC5) -> GND
- D1 pad 1: Net-(D1-K) -> /ROWM
- D18 pad 1: /ROW1 -> /ROW0
- D19 pad 1: /ROW1 -> /ROW0
- D2 pad 1: Net-(D2-K) -> /ROWM
- D20 pad 1: /ROW1 -> /ROW0
- D21 pad 1: /ROW1 -> /ROW0
- D22 pad 1: /ROW1 -> /ROW0
- D23 pad 1: /ROW1 -> /ROW0
- D24 pad 1: /ROW1 -> /ROW0
- D25 pad 1: /ROW1 -> /ROWM
- D26 pad 1: /ROW1 -> /ROWM
- D27 pad 1: /ROW1 -> /ROWM
- D28 pad 1: /ROW1 -> /ROWM
- D3 pad 1: /ROW0 -> /ROWM
- D32 pad 1: /ROW2 -> /ROW1
- D33 pad 1: /ROW2 -> /ROW1
- D34 pad 1: /ROW2 -> /ROW1
- D35 pad 1: /ROW2 -> /ROW1
- D36 pad 1: /ROW2 -> /ROW1
- D37 pad 1: /ROW2 -> /ROW1
- D38 pad 1: /ROW2 -> /ROW1
- D39 pad 1: /ROW2 -> /ROW1
- D4 pad 1: /ROW0 -> /ROWM
- D40 pad 1: /ROW2 -> /ROW1
- D41 pad 1: /ROW2 -> /ROW1
- D42 pad 1: /ROW2 -> /ROW1
- D43 pad 1: /ROW2 -> /ROW1
- D44 pad 1: /ROW2 -> /ROW1
- D45 pad 1: /ROW3 -> /ROW1
- D46 pad 1: /ROW3 -> /ROW1
- D47 pad 1: /ROW3 -> /ROW1
- D48 pad 1: /ROW3 -> /ROW1
- D49 pad 1: /ROW3 -> /ROW1
- D5 pad 1: /ROW0 -> /ROWM
- D50 pad 1: /ROW3 -> /ROW1
- D51 pad 1: /ROW3 -> /ROW2
- D52 pad 1: /ROW3 -> /ROW2
- D53 pad 1: /ROW3 -> /ROW2
- D54 pad 1: /ROW3 -> /ROW2
- D55 pad 1: /ROW3 -> /ROW2
- D56 pad 1: /ROW3 -> /ROW2
- D57 pad 1: /ROW3 -> /ROW2
- D58 pad 1: /ROW4 -> /ROW2
- D59 pad 1: /ROW4 -> /ROW2
- D6 pad 1: /ROW0 -> /ROWM
- D60 pad 1: /ROW4 -> /ROW2
- D61 pad 1: /ROW4 -> /ROW2
- D62 pad 1: /ROW4 -> /ROW2
- D63 pad 1: /ROW4 -> /ROW2
- D64 pad 1: /ROW4 -> /ROW2
- D65 pad 1: /ROW4 -> /ROW2
- D7 pad 1: /ROW0 -> /ROWM
- D8 pad 1: /ROW0 -> /ROWM
- J1 pad 1: /VBUS -> /DB_SWDCLK
- J1 pad 2: /USB_D- -> /DB_SWO
- J1 pad 3: /USB_D+ -> unconnected-(J1-Pin_3-Pad3)
- J1 pad 4: GND -> unconnected-(J1-Pin_4-Pad4)
- J3 pad 1: /DB_SWDCLK -> /VOL_A
- J3 pad 2: /DB_SWO -> /VOL_C
- J3 pad 3: unconnected-(J3-Pin_3-Pad3) -> /VOL_B
- J3 pad 4: unconnected-(J3-Pin_4-Pad4) -> GND
- J4 pad A4: /VBUS -> +5V
- J5 pad 1: Net-(J5-Pin_1) -> +5V
- J5 pad 2: /DB_SWDIO -> /USB_D-
- J5 pad 3: /~{nReset} -> /USB_D+
- J5 pad 4: /DB_SWDCLK -> GND
- JP1 pad 2: Net-(J5-Pin_1) -> Net-(J2-Pin_1)
- L1 pad 1: Net-(U3-ANT) -> Net-(U1-DEC4)
- L1 pad 2: Net-(C11-Pad1) -> Net-(L1-Pad2)
- L2 pad 1: GND -> /VDD_nRF
- L2 pad 2: GNDPWR -> Net-(U1-DCCH)
- L3 pad 1: Net-(L3-Pad1) -> Net-(L1-Pad2)
- L3 pad 2: Net-(U3-DCC) -> Net-(U1-DCC)
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Routing:
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- added copper zone on B.Cu, net +5V
- removed copper zone on B.Cu, net /VBUS
- removed copper zone on B.Cu, net GND
- removed copper zone on F.Cu, net GND
Other:
- board size 284.7 x 94.2 mm -> 458.8 x 145.3 mm
- board text removed: "3V3"
- board text removed: "BLE"
- board text removed: "CLK"
- board text removed: "Designed by Sris"
- board text removed: "Enabled"
- board text removed: "GND"
- board text removed: "IO"
- board text removed: "Logo Credits : VK"
- board text removed: "RST"
- board text removed: "SWO"
- board text removed: "TR-60"
- board text removed: "Version 2.0"
- board text removed: "X"

Commit message: Status LEDs
Parts:
- C1, C10, C100, C101, C102, C103, C104, C105, C106, C107, C108, C109, C11, C110, C111, C112, C113, C114, C115, C116, C117, C118, C119, C12, C120, C121, C13, C14, C15, C16, C17, C18, C19, C2, C20, C21, C22, C23, C24, C25, C26, C27, C28, C29, C3, C30, C31, C32, C33, C34, C35, C36, C37, C38, C39, C4, C40, C41, C42, C43, C44, C45, C46, C47, C48, C49, C5, C50, C51, C52, C53, C54, C55, C56, C57, C58, C59, C6, C60, C61, C62, C63, C64, C65, C66, C67, C68, C69, C7, C70, C71, C72, C73, C74, C75, C76, C77, C78, C79, C8, C80, C81, C82, C83, C84, C85, C86, C87, C88, C89, C9, C90, C91, C92, C93, C94, C95, C96, C97, C98, C99: footprint Capacitor_SMD:C_0402_1005Metric -> keyboard:C_0402_1005Metric
- D1, D10, D100, D101, D102, D103, D104, D105, D106, D107, D108, D109, D11, D110, D111, D112, D113, D114, D115, D116, D117, D118, D119, D12, D120, D121, D13, D14, D15, D16, D17, D18, D19, D2, D20, D21, D22, D23, D24, D25, D26, D27, D28, D29, D3, D30, D31, D32, D33, D34, D35, D36, D37, D38, D39, D4, D40, D41, D42, D43, D44, D45, D46, D47, D48, D49, D5, D50, D51, D52, D53, D54, D55, D56, D57, D58, D59, D6, D60, D61, D62, D63, D64, D65, D66, D67, D68, D69, D7, D70, D71, D72, D73, D74, D75, D76, D77, D78, D79, D8, D80, D81, D82, D83, D84, D85, D86, D87, D88, D89, D9, D90, D91, D92, D93, D94, D95, D96, D97, D98, D99: footprint Diode_SMD:D_SOD-123F -> keyboard:D_SOD-123F
- LED1, LED10, LED100, LED101, LED102, LED103, LED104, LED105, LED106, LED107, LED108, LED109, LED11, LED110, LED111, LED112, LED113, LED114, LED115, LED116, LED117, LED118, LED119, LED12, LED120, LED121, LED13, LED14, LED15, LED16, LED17, LED18, LED19, LED2, LED20, LED21, LED22, LED23, LED24, LED25, LED26, LED27, LED28, LED29, LED3, LED30, LED31, LED32, LED33, LED34, LED35, LED36, LED37, LED38, LED39, LED4, LED40, LED41, LED42, LED43, LED44, LED45, LED46, LED47, LED48, LED49, LED5, LED50, LED51, LED52, LED53, LED54, LED55, LED56, LED57, LED58, LED59, LED6, LED60, LED61, LED62, LED63, LED64, LED65, LED66, LED67, LED68, LED69, LED7, LED70, LED71, LED72, LED73, LED74, LED75, LED76, LED77, LED78, LED79, LED8, LED80, LED81, LED82, LED83, LED84, LED85, LED86, LED87, LED88, LED89, LED9, LED90, LED91, LED92, LED93, LED94, LED95, LED96, LED97, LED98, LED99: footprint LED_SMD:LED_WS2812B_PLCC4_5.0x5.0mm_P3.2mm -> keyboard:LED_WS2812B-2020_PLCC4_2.0x2.0mm
- moved SW1 242.1 mm to (-111.4, 157.5)
Connections:
- U1 pad AC11: /COL16 -> /COL17
- U1 pad AC15: /COL15 -> /COL16
- U1 pad AC17: /COL14 -> /COL15
- U1 pad AC19: /COL13 -> /COL14
- U1 pad AC9: /COL17 -> /COL18
- U1 pad AD12: /~{nReset} -> /COL00
- U1 pad AD16: /COL01 -> /COL02
- U1 pad AD18: /COL12 -> /COL13
- U1 pad AD20: /COL00 -> /COL01
- U1 pad B13: /COL20 -> /MCU_RGB
- U1 pad G1: /COL04 -> /COL05
- U1 pad J24: /COL11 -> /COL12
- U1 pad K2: /MCU_RGB -> /RGB_ENABLE
- U1 pad L1: /COL02 -> /COL03
- U1 pad L24: /COL10 -> /COL11
- U1 pad M2: /COL19 -> /COL20
- U1 pad N1: /COL03 -> /COL04
- U1 pad P2: unconnected-(U1-P1.08-PadP2) -> /~{nReset}
- U1 pad R1: /COL08 -> /COL09
- U1 pad R24: /COL07 -> /COL08
- U1 pad T2: /COL18 -> /COL19
- U1 pad U1: /COL09 -> /COL10
- U1 pad U24: /COL06 -> /COL07
- U1 pad W24: /COL05 -> /COL06
