File: zmk-g915.kicad_pcb (KiCad board)
At the start: 2 copper layers, 458.6 x 143.2 mm, 611 parts, among them J1 Prog_conn, J2 Tag connect TC2030-CTX, J3 53047-0460, J4 TYPE-C-31-M12_13, J5 JST-4-pin, Q1 Q_NMOS, Q2 Q_NMOS, Q3 Q_NMOS, SW1 Reset Switch, U1 nRF52840-QIAA-R/nRF52833-QIAA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, U2 TPD4E05U06DQAR, U3 BQ24074RGTR, U4 BQ24074RGTR, Y1 32.768kHz, Y2 32MHz

Commit message: Minor pcb layout changes. Add matrix led drivers
Parts:
- moved MX1 1.10 mm to (88.8, 247.1)
- moved MX2 1.10 mm to (106.8, 247.1)
- moved MX4 1.10 mm to (142.8, 247.1)
- moved MX5 1.10 mm to (177.7, 247.1)
- moved MX6 1.10 mm to (195.7, 247.1)
- moved MX3 1.10 mm to (124.8, 247.1)
- moved MX7 1.10 mm to (213.7, 247.1)
- moved MX8 1.10 mm to (231.7, 247.1)
- moved REF** 0.05 mm to (445.1, 303.8)
Other:
- outline, holes or cut-outs redrawn
