File: switch_matrix.kicad_sch (KiCad schematic)
At the start: 0 parts

Commit message: Switch to matrix RGB LED
Other:
- removed sheet K_0
- removed sheet K_1
- removed sheet K_2
- removed sheet K_3
- removed sheet K_4
- removed sheet K_5
- removed sheet K_6
- removed sheet K_7
- removed sheet K_8
- removed sheet K_9
- removed sheet K_A
- removed sheet K_Apostrophe
- removed sheet K_B
- removed sheet K_Backslash
- removed sheet K_Backspace
- removed sheet K_Bluetooth
- removed sheet K_Brightness
- removed sheet K_C
- removed sheet K_CAPS
- removed sheet K_Comma
- removed sheet K_D
- removed sheet K_DEL
- removed sheet K_DOWN
- removed sheet K_E
- removed sheet K_END
- removed sheet K_ENTER
- removed sheet K_ESC
- removed sheet K_Equals
- removed sheet K_F
- removed sheet K_F1
- removed sheet K_F10
- removed sheet K_F11
- removed sheet K_F12
- removed sheet K_F2
- removed sheet K_F3
- removed sheet K_F4
- removed sheet K_F5
- removed sheet K_F6
- removed sheet K_F7
- removed sheet K_F8
- removed sheet K_F9
- removed sheet K_G
- removed sheet K_G1
- removed sheet K_G2
- removed sheet K_G3
- removed sheet K_G4
- removed sheet K_G5
- removed sheet K_GameMode
- removed sheet K_H
- removed sheet K_HOME
- removed sheet K_I
- removed sheet K_INS
- removed sheet K_J
- removed sheet K_K
- removed sheet K_L
- removed sheet K_LALT
- removed sheet K_LBracket
- removed sheet K_LCTRL
- removed sheet K_LEFT
- removed sheet K_LSHIFT
- removed sheet K_LWin
- removed sheet K_M
- removed sheet K_M1
- removed sheet K_M2
- removed sheet K_M3
- removed sheet K_MR
- removed sheet K_Menu
- removed sheet K_Minus
- removed sheet K_Mute
- removed sheet K_N
- removed sheet K_Next
- removed sheet K_O
- removed sheet K_P
- removed sheet K_PAUSE
- removed sheet K_PGDN
- removed sheet K_PGUP
- removed sheet K_PRTSC
- removed sheet K_Period
- removed sheet K_Play
- removed sheet K_Prev
- removed sheet K_Q
- removed sheet K_R
- removed sheet K_RALT
- removed sheet K_RBracket
- removed sheet K_RCTRL
- removed sheet K_RIGHT
- removed sheet K_RSHIFT
- removed sheet K_RWIN
- removed sheet K_S
- removed sheet K_SCRLK
- removed sheet K_Semicolon
- removed sheet K_Slash
- removed sheet K_Space
- removed sheet K_T
- removed sheet K_TAB
- removed sheet K_Tilde
- removed sheet K_U
- removed sheet K_UP
- removed sheet K_V
- removed sheet K_W
- removed sheet K_Wireless
- removed sheet K_X
- removed sheet K_Y
- removed sheet K_Z
- removed sheet K_np0
- removed sheet K_np1
- removed sheet K_np2
- removed sheet K_np3
- removed sheet K_np4
- removed sheet K_np5
- removed sheet K_np6
- removed sheet K_np7
- removed sheet K_np8
- removed sheet K_np9
- removed sheet K_npAsterisk
- removed sheet K_npDecimal
- removed sheet K_npEnter
- removed sheet K_npMinus
- removed sheet K_npNUM
- removed sheet K_npPlus
- removed sheet K_npSlash
- added sheet 0 (key.kicad_sch)
- added sheet 1 (key.kicad_sch)
- added sheet 2 (key.kicad_sch)
- added sheet 3 (key.kicad_sch)
- added sheet 4 (key.kicad_sch)
- added sheet 5 (key.kicad_sch)
- added sheet 6 (key.kicad_sch)
- added sheet 7 (key.kicad_sch)
- added sheet 8 (key.kicad_sch)
- added sheet 9 (key.kicad_sch)
- added sheet A (key.kicad_sch)
- added sheet Apostrophe (key.kicad_sch)
- added sheet B (key.kicad_sch)
- added sheet Backslash (key.kicad_sch)
- added sheet Backspace (key.kicad_sch)
- added sheet Bluetooth (key-mem.kicad_sch)
- added sheet Brightness (key-mem.kicad_sch)
- added sheet C (key.kicad_sch)
- added sheet CAPS (key.kicad_sch)
- added sheet Comma (key.kicad_sch)
- added sheet D (key.kicad_sch)
- added sheet DEL (key.kicad_sch)
- added sheet Dash (key.kicad_sch)
- added sheet Down (key.kicad_sch)
- added sheet E (key.kicad_sch)
- added sheet END (key.kicad_sch)
- added sheet ENTER (key.kicad_sch)
- added sheet ESC (key.kicad_sch)
- added sheet Equals (key.kicad_sch)
- added sheet F (key.kicad_sch)
- added sheet F1 (key.kicad_sch)
- added sheet F10 (key.kicad_sch)
- added sheet F11 (key.kicad_sch)
- added sheet F12 (key.kicad_sch)
- added sheet F2 (key.kicad_sch)
- added sheet F3 (key.kicad_sch)
- added sheet F4 (key.kicad_sch)
- added sheet F5 (key.kicad_sch)
- added sheet F6 (key.kicad_sch)
- added sheet F7 (key.kicad_sch)
- added sheet F8 (key.kicad_sch)
- added sheet F9 (key.kicad_sch)
- added sheet G (key.kicad_sch)
- added sheet G1 (key.kicad_sch)
- added sheet G2 (key.kicad_sch)
- added sheet G3 (key.kicad_sch)
- added sheet G4 (key.kicad_sch)
- added sheet G5 (key.kicad_sch)
- added sheet GameMode (key-mem.kicad_sch)
- added sheet H (key.kicad_sch)
- added sheet HOME (key.kicad_sch)
- added sheet I (key.kicad_sch)
- added sheet INS (key.kicad_sch)
- added sheet J (key.kicad_sch)
- added sheet K (key.kicad_sch)
- added sheet L (key.kicad_sch)
- added sheet LBracket (key.kicad_sch)
- added sheet Left (key.kicad_sch)
- added sheet M (key.kicad_sch)
- added sheet M1 (key-mem.kicad_sch)
- added sheet M2 (key-mem.kicad_sch)
- added sheet M3 (key-mem.kicad_sch)
- added sheet MR (key-mem.kicad_sch)
- added sheet Menu (key.kicad_sch)
- added sheet Mute (key-mem.kicad_sch)
- added sheet N (key.kicad_sch)
- added sheet Next (key-mem.kicad_sch)
- added sheet O (key.kicad_sch)
- added sheet P (key.kicad_sch)
- added sheet PAUSE (key.kicad_sch)
- added sheet PGDN (key.kicad_sch)
- added sheet PGUP (key.kicad_sch)
- added sheet PRTSC (key.kicad_sch)
- added sheet Period (key.kicad_sch)
- added sheet PlayPause (key-mem.kicad_sch)
- added sheet Previous (key-mem.kicad_sch)
- added sheet Q (key.kicad_sch)
- added sheet R (key.kicad_sch)
- added sheet RBracket (key.kicad_sch)
- added sheet Right (key.kicad_sch)
- added sheet S (key.kicad_sch)
- added sheet SCRLK (key.kicad_sch)
- added sheet Semicolon (key.kicad_sch)
- added sheet Slash (key.kicad_sch)
- added sheet Space (key.kicad_sch)
- added sheet T (key.kicad_sch)
- added sheet TAB (key.kicad_sch)
- added sheet Tilde (key.kicad_sch)
- added sheet U (key.kicad_sch)
- added sheet Up (key.kicad_sch)
- added sheet V (key.kicad_sch)
- added sheet W (key.kicad_sch)
- added sheet Wireless (key-mem.kicad_sch)
- added sheet X (key.kicad_sch)
- added sheet Y (key.kicad_sch)
- added sheet Z (key.kicad_sch)
- added sheet lALT (key.kicad_sch)
- added sheet lCTRL (key.kicad_sch)
- added sheet lSHIFT (key.kicad_sch)
- added sheet lWIN (key.kicad_sch)
- added sheet np0 (key.kicad_sch)
- added sheet np1 (key.kicad_sch)
- added sheet np2 (key.kicad_sch)
- added sheet np3 (key.kicad_sch)
- added sheet np4 (key.kicad_sch)
- added sheet np5 (key.kicad_sch)
- added sheet np6 (key.kicad_sch)
- added sheet np7 (key.kicad_sch)
- added sheet np8 (key.kicad_sch)
- added sheet np9 (key.kicad_sch)
- added sheet npAsterisk (key.kicad_sch)
- added sheet npDecimal (key.kicad_sch)
- added sheet npENTER (key.kicad_sch)
- added sheet npMinus (key.kicad_sch)
- added sheet npNUM (key.kicad_sch)
- added sheet npPlus (key.kicad_sch)
- added sheet npSlash (key.kicad_sch)
- added sheet rALT (key.kicad_sch)
- added sheet rCTRL (key.kicad_sch)
- added sheet rSHIFT (key.kicad_sch)
- added sheet rWIN (key.kicad_sch)

Commit message: led matrix sheet
Other:
- company: HW-tinkerers -> (none)
