File: USB_power.kicad_sch (KiCad schematic)
At the start: 24 parts, among them J4 TYPE-C-31-M12_13, J5 JST-4-pin, Q2 Q_NMOS, U2 TPD4E05U06DQAR, U3 BQ24074RGTR

Commit message: led matrix work
Parts:
- C21: value 4u7F -> 4.7uF
Changed lines of the file:
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@@
 	)
 	(hierarchical_label "USB_D+"
-		(shape bidirectional)
+		(shape passive)
 		(at 81.28 190.5 0)
 		(effects
@@
 	)
 	(hierarchical_label "USB_D-"
-		(shape bidirectional)
+		(shape passive)
 		(at 81.28 186.69 0)
 		(effects
@@
 	)
 	(hierarchical_label "CHG_OUT"
-		(shape output)
+		(shape passive)
 		(at 40.64 190.5 0)
 		(effects
@@
 	)
 	(hierarchical_label "VBATT_nRF"
-		(shape output)
+		(shape passive)
 		(at 115.57 186.69 0)
 		(effects
@@
 	)
 	(hierarchical_label "VBUS"
-		(shape output)
+		(shape passive)
 		(at 40.64 186.69 0)
 		(effects
@@
 			)
 		)
-		(property "Value" "4u7F"
+		(property "Value" "4.7uF"
 			(at 95.25 132.08 0)
 			(effects
