File: redragon-k618-pro/rgb_led.kicad_sch (KiCad schematic)
At the start: 1 part

Commit message: g915 pcb and k618 pcb and matrix sch work
Parts:
- LED1: footprint (none) -> LED_SMD:LED_WS2812B-2020_PLCC4_2.0x2.0mm
