File: redragon-k618-pro/zmk-k618.kicad_pcb (KiCad board)
At the start: 2 copper layers, 431.9 x 138.7 mm, 590 parts, among them J1 Prog_conn, J2 Tag connect TC2030-CTX, J3 53047-0460, J4 TYPE-C-31-M12_13, J5 JST-4-pin, Q1 Q_NMOS, Q3 Q_NMOS, SW1 Reset Switch, U1 nRF52840-QIAA-R/nRF52833-QIAA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, U2 SN74AHCT1G125, U3 TPD4E05U06DQAR, U4 BQ24074RGTR, Y1 32.768kHz, Y2 32MHz

Commit message: g915 pcb key spacing work
Parts:
- moved C29 199.7 mm to (526.8, 89.5)
- moved D16 199.7 mm to (265.7, 92.6)
- moved D17 199.7 mm to (284.7, 92.6)
- moved D18 199.7 mm to (303.7, 92.6)
- moved D19 199.7 mm to (322.7, 92.6)
- moved D20 199.7 mm to (351.2, 92.6)
- moved D37 199.7 mm to (256.2, 114.5)
- moved D38 199.7 mm to (275.2, 114.5)
- moved D39 199.7 mm to (294.2, 114.5)
- moved D40 199.7 mm to (313.2, 114.5)
- moved D41 199.7 mm to (332.2, 114.5)
- moved D42 199.7 mm to (351.2, 114.5)
- moved LED29 199.7 mm to (526.8, 89.5)
- moved MX29 199.7 mm to (526.8, 89.5)
- moved C1 199.7 mm to (155.6, 70.5)
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
Commit message: g915 pcb and k618 pcb and matrix sch work
Parts:
- C1, C16, C18, C21: value 100nF -> 4u7F
- C11: value 100nF -> 820pF
- C12: value 100nF -> 100pF
- C13: value 100nF -> DNP
- C17: value 100nF -> 1pF
- C19: value 100nF -> 1.2pF
- C2, C3, C8, C9: value 100nF -> 8pF
- C20, C4, C6: value 100nF -> 1uF
- D119, D120, D121: value B140S1F-7 -> LED
- LED1, LED10, LED100, LED101, LED102, LED103, LED104, LED105, LED106, LED107, LED108, LED109, LED11, LED110, LED111, LED112, LED113, LED114, LED115, LED116, LED117, LED118, LED12, LED13, LED14, LED15, LED16, LED17, LED18, LED19, LED2, LED20, LED21, LED22, LED23, LED24, LED25, LED26, LED27, LED28, LED29, LED3, LED30, LED31, LED32, LED33, LED34, LED35, LED36, LED37, LED38, LED39, LED4, LED40, LED41, LED42, LED43, LED44, LED45, LED46, LED47, LED48, LED49, LED5, LED50, LED51, LED52, LED53, LED54, LED55, LED56, LED57, LED58, LED59, LED6, LED60, LED61, LED62, LED63, LED64, LED65, LED66, LED67, LED68, LED69, LED7, LED70, LED71, LED72, LED73, LED74, LED75, LED76, LED77, LED78, LED79, LED8, LED80, LED81, LED82, LED83, LED84, LED85, LED86, LED87, LED88, LED89, LED9, LED90, LED91, LED92, LED93, LED94, LED95, LED96, LED97, LED98, LED99: value WS2812B -> LED_ARGB; footprint keyboard:LED_WS2812B-2020_PLCC4_2.0x2.0mm -> LED_SMD:LED_WS2812B-2020_PLCC4_2.0x2.0mm
- MX1, MX2, MX27, MX28, MX3, MX4, MX5, MX6, MX7, MX8: footprint G915:Membrane-G915 -> K618:membrane
- MX10, MX29, MX30, MX9: footprint key-switches:SW_Gateron_LowProfile_HotSwap_PTH -> K618:membrane
- MX25, MX26: footprint G915:Membrane-G915 -> key-switches:SW_Gateron_LowProfile_HotSwap_PTH
- R10: value 5k1 -> 10k
- R11: value 1k2 -> 5k1
- R12: value 8k2 -> 5k1
- R13: value 5k1 -> R_US
- R14: value R_US -> 1k2
- R15: value 10k -> VAL
- R16: value 10k -> 5k1
- R17: value 10k -> R_US
- R19, R22: value R_US -> 10k
- R8: value 100 -> R_US
- R9: value 5k1 -> 100
- U2: value SN74AHCT1G125 -> TPD4E05U06DQAR
- U3: value TPD4E05U06DQAR -> BQ24074RGTR
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Connections:
- C1 pad 1: +5V -> /VDD_nRF
- C10 pad 1: +5V -> /VDD_nRF
- C11 pad 1: +5V -> GND
- C11 pad 2: GND -> Net-(U1-DEC5)
- C12 pad 1: +5V -> GND
- C12 pad 2: GND -> Net-(U1-DEC3)
- C13 pad 1: +5V -> GND
- C13 pad 2: GND -> Net-(U1-DEC2)
- C14 pad 1: +5V -> GND
- C14 pad 2: GND -> Net-(U1-DEC1)
- C15 pad 1: +5V -> /VDD_nRF
- C16 pad 1: +5V -> Net-(U1-DECUSB)
- C17 pad 1: +5V -> Net-(U1-ANT)
- C19 pad 1: +5V -> Net-(C19-Pad1)
- C2 pad 1: +5V -> GND
- C2 pad 2: GND -> Net-(U1-XC2)
- C21 pad 1: +5V -> /USB and Power management/V_BATT
- C22 pad 1: +5V -> /VBATT_nRF
- C3 pad 1: +5V -> GND
- C3 pad 2: GND -> Net-(U1-P0.00/XL1)
- C4 pad 1: +5V -> GND
- C4 pad 2: GND -> /VDD_nRF
- C5 pad 1: +5V -> GND
- C5 pad 2: GND -> Net-(U1-DEC4)
- C6 pad 1: +5V -> Net-(U1-DEC4)
- C7 pad 1: +5V -> /VDD_nRF
- C8 pad 1: +5V -> GND
- C8 pad 2: GND -> Net-(U1-P0.01/XL2)
- C9 pad 1: +5V -> GND
- C9 pad 2: GND -> Net-(U1-XC1)
- D1 pad 1: /ROWM -> /switch_matrix/ROWM
- D10 pad 1: /ROW0 -> /switch_matrix/ROWM
- D100 pad 1: /ROW4 -> /switch_matrix/ROW4
- D101 pad 1: /ROW4 -> /switch_matrix/ROW4
- D102 pad 1: /ROW4 -> /switch_matrix/ROW4
- D103 pad 1: /ROW4 -> /switch_matrix/ROW4
- D104 pad 1: /ROW4 -> /switch_matrix/ROW4
- D105 pad 1: /ROW4 -> /switch_matrix/ROW4
- D106 pad 1: /ROW4 -> /switch_matrix/ROW5
- D107 pad 1: /ROW4 -> /switch_matrix/ROW5
- D108 pad 1: /ROW5 -> /switch_matrix/ROW5
- D109 pad 1: /ROW5 -> /switch_matrix/ROW5
- D11 pad 1: /ROW0 -> /switch_matrix/ROW0
- D110 pad 1: /ROW5 -> /switch_matrix/ROW5
- D111 pad 1: /ROW5 -> /switch_matrix/ROW5
- D112 pad 1: /ROW5 -> /switch_matrix/ROW5
- D113 pad 1: /ROW5 -> /switch_matrix/ROW5
- D114 pad 1: /ROW5 -> /switch_matrix/ROW5
- D115 pad 1: /ROW5 -> /switch_matrix/ROW5
- D116 pad 1: /ROW5 -> /switch_matrix/ROW5
- D117 pad 1: /ROW5 -> /switch_matrix/ROW5
- D118 pad 1: /ROW5 -> /switch_matrix/ROW5
- D119 pad 1: /ROW5 -> Net-(D119-K)
- D12 pad 1: /ROW0 -> /switch_matrix/ROW0
- D120 pad 1: /ROW5 -> Net-(D120-K)
- D121 pad 1: /ROW5 -> Net-(D121-K)
- D13 pad 1: /ROW0 -> /switch_matrix/ROW0
- D14 pad 1: /ROW0 -> /switch_matrix/ROW0
- D15 pad 1: /ROW0 -> /switch_matrix/ROW0
- D16 pad 1: /ROW0 -> /switch_matrix/ROW0
- D17 pad 1: /ROW0 -> /switch_matrix/ROW0
- D18 pad 1: /ROW0 -> /switch_matrix/ROW0
- D19 pad 1: /ROW0 -> /switch_matrix/ROW0
- D2 pad 1: /ROWM -> /switch_matrix/ROWM
- D20 pad 1: /ROW0 -> /switch_matrix/ROW0
- D21 pad 1: /ROW0 -> /switch_matrix/ROW0
- D22 pad 1: /ROW0 -> /switch_matrix/ROW0
- D23 pad 1: /ROW0 -> /switch_matrix/ROW0
- D24 pad 1: /ROW0 -> /switch_matrix/ROW0
- D25 pad 1: /ROWM -> /switch_matrix/ROW0
- D26 pad 1: /ROWM -> /switch_matrix/ROW0
- D27 pad 1: /ROWM -> /switch_matrix/ROWM
- D28 pad 1: /ROWM -> /switch_matrix/ROWM
- D29 pad 1: /ROW1 -> /switch_matrix/ROWM
- D3 pad 1: /ROWM -> /switch_matrix/ROWM
- D30 pad 1: /ROW1 -> /switch_matrix/ROWM
- D31 pad 1: /ROW1 -> /switch_matrix/ROW1
- D32 pad 1: /ROW1 -> /switch_matrix/ROW1
- D33 pad 1: /ROW1 -> /switch_matrix/ROW1
- D34 pad 1: /ROW1 -> /switch_matrix/ROW1
- D35 pad 1: /ROW1 -> /switch_matrix/ROW1
- D36 pad 1: /ROW1 -> /switch_matrix/ROW1
- D37 pad 1: /ROW1 -> /switch_matrix/ROW1
- D38 pad 1: /ROW1 -> /switch_matrix/ROW1
- D39 pad 1: /ROW1 -> /switch_matrix/ROW1
- D4 pad 1: /ROWM -> /switch_matrix/ROWM
- D40 pad 1: /ROW1 -> /switch_matrix/ROW1
- D41 pad 1: /ROW1 -> /switch_matrix/ROW1
- D42 pad 1: /ROW1 -> /switch_matrix/ROW1
- D43 pad 1: /ROW1 -> /switch_matrix/ROW1
- D44 pad 1: /ROW1 -> /switch_matrix/ROW1
- D45 pad 1: /ROW1 -> /switch_matrix/ROW1
- D46 pad 1: /ROW1 -> /switch_matrix/ROW1
- D47 pad 1: /ROW1 -> /switch_matrix/ROW1
- D48 pad 1: /ROW1 -> /switch_matrix/ROW1
- D49 pad 1: /ROW1 -> /switch_matrix/ROW1
- D5 pad 1: /ROWM -> /switch_matrix/ROWM
- D50 pad 1: /ROW1 -> /switch_matrix/ROW1
- D51 pad 1: /ROW2 -> /switch_matrix/ROW1
- D52 pad 1: /ROW2 -> /switch_matrix/ROW2
- D53 pad 1: /ROW2 -> /switch_matrix/ROW2
- D54 pad 1: /ROW2 -> /switch_matrix/ROW2
- D55 pad 1: /ROW2 -> /switch_matrix/ROW2
- D56 pad 1: /ROW2 -> /switch_matrix/ROW2
- D57 pad 1: /ROW2 -> /switch_matrix/ROW2
- D58 pad 1: /ROW2 -> /switch_matrix/ROW2
- D59 pad 1: /ROW2 -> /switch_matrix/ROW2
- D6 pad 1: /ROWM -> /switch_matrix/ROWM
- D60 pad 1: /ROW2 -> /switch_matrix/ROW2
- D61 pad 1: /ROW2 -> /switch_matrix/ROW2
- D62 pad 1: /ROW2 -> /switch_matrix/ROW2
- D63 pad 1: /ROW2 -> /switch_matrix/ROW2
- D64 pad 1: /ROW2 -> /switch_matrix/ROW2
- D65 pad 1: /ROW2 -> /switch_matrix/ROW2
- D66 pad 1: /ROW2 -> /switch_matrix/ROW2
- D67 pad 1: /ROW2 -> /switch_matrix/ROW2
- D68 pad 1: /ROW2 -> /switch_matrix/ROW2
- D69 pad 1: /ROW2 -> /switch_matrix/ROW2
- D7 pad 1: /ROWM -> /switch_matrix/ROWM
- D70 pad 1: /ROW2 -> /switch_matrix/ROW2
- D71 pad 1: /ROW2 -> /switch_matrix/ROW2
- D72 pad 1: /ROW2 -> /switch_matrix/ROW2
- D73 pad 1: /ROW3 -> /switch_matrix/ROW3
- D74 pad 1: /ROW3 -> /switch_matrix/ROW3
- D75 pad 1: /ROW3 -> /switch_matrix/ROW3
- D76 pad 1: /ROW3 -> /switch_matrix/ROW3
- D77 pad 1: /ROW3 -> /switch_matrix/ROW3
- D78 pad 1: /ROW3 -> /switch_matrix/ROW3
- D79 pad 1: /ROW3 -> /switch_matrix/ROW3
- D8 pad 1: /ROWM -> /switch_matrix/ROWM
- D80 pad 1: /ROW3 -> /switch_matrix/ROW3
- D81 pad 1: /ROW3 -> /switch_matrix/ROW3
- D82 pad 1: /ROW3 -> /switch_matrix/ROW3
- D83 pad 1: /ROW3 -> /switch_matrix/ROW3
- D84 pad 1: /ROW3 -> /switch_matrix/ROW3
- D85 pad 1: /ROW3 -> /switch_matrix/ROW3
- D86 pad 1: /ROW3 -> /switch_matrix/ROW3
- D87 pad 1: /ROW3 -> /switch_matrix/ROW3
- D88 pad 1: /ROW3 -> /switch_matrix/ROW3
- D89 pad 1: /ROW3 -> /switch_matrix/ROW4
- D9 pad 1: /ROW0 -> /switch_matrix/ROWM
- D90 pad 1: /ROW4 -> /switch_matrix/ROW4
- D91 pad 1: /ROW4 -> /switch_matrix/ROW4
- D92 pad 1: /ROW4 -> /switch_matrix/ROW4
- D93 pad 1: /ROW4 -> /switch_matrix/ROW4
- D94 pad 1: /ROW4 -> /switch_matrix/ROW4
- D95 pad 1: /ROW4 -> /switch_matrix/ROW4
- D96 pad 1: /ROW4 -> /switch_matrix/ROW4
- D97 pad 1: /ROW4 -> /switch_matrix/ROW4
- D98 pad 1: /ROW4 -> /switch_matrix/ROW4
- D99 pad 1: /ROW4 -> /switch_matrix/ROW4
- L4 pad 2: Net-(C140-Pad1) -> Net-(C19-Pad1)
- L5 pad 1: Net-(C140-Pad1) -> Net-(C19-Pad1)
- LED1 pad 1: +5V -> /rgb-led_matrix/C1.4
- LED1 pad 2: /switch_matrix/K_M1/DOUT -> /rgb-led_matrix/S1.1
- LED1 pad 3: GND -> /rgb-led_matrix/S1.2
- LED1 pad 4: /RGB_DIN -> /rgb-led_matrix/S1.3
- LED10 pad 1: +5V -> /rgb-led_matrix/C1.12
- LED10 pad 2: /switch_matrix/K_ESC/DIN -> /rgb-led_matrix/S1.1
- LED10 pad 3: GND -> /rgb-led_matrix/S1.2
- LED10 pad 4: /switch_matrix/K_F1/DIN -> /rgb-led_matrix/S1.3
- LED100 pad 1: +5V -> /rgb-led_matrix/C2.5
- LED100 pad 2: /switch_matrix/K_Comma/DIN -> /rgb-led_matrix/S2.7
- LED100 pad 3: GND -> /rgb-led_matrix/S2.8
- LED100 pad 4: /switch_matrix/K_Period/DIN -> /rgb-led_matrix/S2.9
- LED101 pad 1: +5V -> /rgb-led_matrix/C2.7
- LED101 pad 2: /switch_matrix/K_Period/DIN -> /rgb-led_matrix/S2.7
- LED101 pad 3: GND -> /rgb-led_matrix/S2.8
- LED101 pad 4: /switch_matrix/K_RSHIFT/DOUT -> /rgb-led_matrix/S2.9
- LED102 pad 1: +5V -> /rgb-led_matrix/np2/AN
- LED102 pad 2: /switch_matrix/K_RSHIFT/DOUT -> /rgb-led_matrix/S2.7
- LED102 pad 3: GND -> /rgb-led_matrix/S2.8
- LED102 pad 4: /switch_matrix/K_RSHIFT/DIN -> /rgb-led_matrix/S2.9
- LED103 pad 1: +5V -> /rgb-led_matrix/np3/AN
- LED103 pad 2: /switch_matrix/K_RSHIFT/DIN -> /rgb-led_matrix/S2.7
- LED103 pad 3: GND -> /rgb-led_matrix/S2.8
- LED103 pad 4: /switch_matrix/K_UP/DIN -> /rgb-led_matrix/S2.9
- LED104 pad 1: +5V -> /rgb-led_matrix/C2.10
- LED104 pad 2: /switch_matrix/K_UP/DIN -> /rgb-led_matrix/S2.4
- LED104 pad 3: GND -> /rgb-led_matrix/S2.5
- LED104 pad 4: /switch_matrix/K_np1/DIN -> /rgb-led_matrix/S2.6
- LED105 pad 1: +5V -> /rgb-led_matrix/C1.2
- LED105 pad 2: /switch_matrix/K_np1/DIN -> /rgb-led_matrix/S1.10
- LED105 pad 3: GND -> /rgb-led_matrix/S1.11
- LED105 pad 4: /switch_matrix/K_np2/DIN -> /rgb-led_matrix/S1.12
- LED106 pad 1: +5V -> /rgb-led_matrix/C1.2
- LED106 pad 2: /switch_matrix/K_np2/DIN -> /rgb-led_matrix/S1.10
- LED106 pad 3: GND -> /rgb-led_matrix/S1.11
- LED106 pad 4: /switch_matrix/K_np3/DIN -> /rgb-led_matrix/S1.12
- LED107 pad 1: +5V -> /rgb-led_matrix/C1.3
- LED107 pad 2: /switch_matrix/RGB_DOUT -> /rgb-led_matrix/S1.10
- LED107 pad 3: GND -> /rgb-led_matrix/S1.11
- LED107 pad 4: /switch_matrix/K_npDecimal/DOUT -> /rgb-led_matrix/S1.12
- LED108 pad 1: +5V -> /rgb-led_matrix/C1.7
- LED108 pad 2: /switch_matrix/K_G5/DOUT -> /rgb-led_matrix/S1.10
- LED108 pad 3: GND -> /rgb-led_matrix/S1.11
- LED108 pad 4: /switch_matrix/K_G4/DOUT -> /rgb-led_matrix/S1.12
- LED109 pad 1: +5V -> /rgb-led_matrix/C1.10
- LED109 pad 2: /switch_matrix/K_LCTRL/DOUT -> /rgb-led_matrix/S1.10
- LED109 pad 3: GND -> /rgb-led_matrix/S1.11
- LED109 pad 4: /switch_matrix/K_G5/DOUT -> /rgb-led_matrix/S1.12
- LED11 pad 1: +5V -> /rgb-led_matrix/C1.2
- LED11 pad 2: /switch_matrix/K_F1/DIN -> /rgb-led_matrix/S1.1
- LED11 pad 3: GND -> /rgb-led_matrix/S1.2
- LED11 pad 4: /switch_matrix/K_F2/DIN -> /rgb-led_matrix/S1.3
- LED110 pad 1: +5V -> /rgb-led_matrix/C1.11
- LED110 pad 2: /switch_matrix/K_LALT/DIN -> /rgb-led_matrix/S1.10
- LED110 pad 3: GND -> /rgb-led_matrix/S1.11
- LED110 pad 4: /switch_matrix/K_LCTRL/DOUT -> /rgb-led_matrix/S1.12
- LED111 pad 1: +5V -> /rgb-led_matrix/C2.1
- LED111 pad 2: /switch_matrix/K_LALT/DOUT -> /rgb-led_matrix/S2.10
- LED111 pad 3: GND -> /rgb-led_matrix/S2.11
- LED111 pad 4: /switch_matrix/K_LALT/DIN -> /rgb-led_matrix/S2.12
- LED112 pad 1: +5V -> /rgb-led_matrix/C2.2
- LED112 pad 2: /switch_matrix/K_RALT/DIN -> /rgb-led_matrix/S2.10
- LED112 pad 3: GND -> /rgb-led_matrix/S2.11
- LED112 pad 4: /switch_matrix/K_LALT/DOUT -> /rgb-led_matrix/S2.12
- LED113 pad 1: +5V -> /rgb-led_matrix/C2.4
- LED113 pad 2: /switch_matrix/K_RALT/DOUT -> /rgb-led_matrix/S2.10
- LED113 pad 3: GND -> /rgb-led_matrix/S2.11
- LED113 pad 4: /switch_matrix/K_RALT/DIN -> /rgb-led_matrix/S2.12
- LED114 pad 1: +5V -> /rgb-led_matrix/C2.5
- LED114 pad 2: /switch_matrix/K_Menu/DIN -> /rgb-led_matrix/S2.10
- LED114 pad 3: GND -> /rgb-led_matrix/S2.11
- LED114 pad 4: /switch_matrix/K_RALT/DOUT -> /rgb-led_matrix/S2.12
- LED115 pad 1: +5V -> /rgb-led_matrix/C2.6
- LED115 pad 2: /switch_matrix/K_Menu/DOUT -> /rgb-led_matrix/S2.10
- LED115 pad 3: GND -> /rgb-led_matrix/S2.11
- LED115 pad 4: /switch_matrix/K_Menu/DIN -> /rgb-led_matrix/S2.12
- LED116 pad 1: +5V -> /rgb-led_matrix/C2.7
- LED116 pad 2: /switch_matrix/K_LEFT/DIN -> /rgb-led_matrix/S2.10
- LED116 pad 3: GND -> /rgb-led_matrix/S2.11
- LED116 pad 4: /switch_matrix/K_Menu/DOUT -> /rgb-led_matrix/S2.12
- LED117 pad 1: +5V -> /rgb-led_matrix/C2.9
- LED117 pad 2: /switch_matrix/K_DOWN/DIN -> /rgb-led_matrix/S2.10
- LED117 pad 3: GND -> /rgb-led_matrix/S2.11
- LED117 pad 4: /switch_matrix/K_LEFT/DIN -> /rgb-led_matrix/S2.12
- LED118 pad 1: +5V -> /rgb-led_matrix/C2.10
- LED118 pad 2: /switch_matrix/K_DOWN/DOUT -> /rgb-led_matrix/S2.7
- LED118 pad 3: GND -> /rgb-led_matrix/S2.8
- LED118 pad 4: /switch_matrix/K_DOWN/DIN -> /rgb-led_matrix/S2.9
- LED12 pad 1: +5V -> /rgb-led_matrix/C1.4
- LED12 pad 2: /switch_matrix/K_F2/DIN -> /rgb-led_matrix/S1.1
- LED12 pad 3: GND -> /rgb-led_matrix/S1.2
- LED12 pad 4: /switch_matrix/K_F3/DIN -> /rgb-led_matrix/S1.3
- LED13 pad 1: +5V -> /rgb-led_matrix/C1.5
- LED13 pad 2: /switch_matrix/K_F3/DIN -> /rgb-led_matrix/S1.1
- LED13 pad 3: GND -> /rgb-led_matrix/S1.2
- LED13 pad 4: /switch_matrix/K_F4/DIN -> /rgb-led_matrix/S1.3
- LED14 pad 1: +5V -> /rgb-led_matrix/C1.6
- LED14 pad 2: /switch_matrix/K_F4/DIN -> /rgb-led_matrix/S1.1
- LED14 pad 3: GND -> /rgb-led_matrix/S1.2
- LED14 pad 4: /switch_matrix/K_F5/DIN -> /rgb-led_matrix/S1.3
- LED15 pad 1: +5V -> /rgb-led_matrix/C1.7
- LED15 pad 2: /switch_matrix/K_F5/DIN -> /rgb-led_matrix/S1.1
- LED15 pad 3: GND -> /rgb-led_matrix/S1.2
- LED15 pad 4: /switch_matrix/K_F6/DIN -> /rgb-led_matrix/S1.3
- LED16 pad 1: +5V -> /rgb-led_matrix/C1.9
- LED16 pad 2: /switch_matrix/K_F6/DIN -> /rgb-led_matrix/S1.1
- LED16 pad 3: GND -> /rgb-led_matrix/S1.2
- LED16 pad 4: /switch_matrix/K_F7/DIN -> /rgb-led_matrix/S1.3
- LED17 pad 1: +5V -> /rgb-led_matrix/C1.10
- LED17 pad 2: /switch_matrix/K_F7/DIN -> /rgb-led_matrix/S1.1
- LED17 pad 3: GND -> /rgb-led_matrix/S1.2
- LED17 pad 4: /switch_matrix/K_F8/DIN -> /rgb-led_matrix/S1.3
- LED18 pad 1: +5V -> /rgb-led_matrix/C1.11
- LED18 pad 2: /switch_matrix/K_F8/DIN -> /rgb-led_matrix/S1.1
- LED18 pad 3: GND -> /rgb-led_matrix/S1.2
- LED18 pad 4: /switch_matrix/K_F10/DOUT -> /rgb-led_matrix/S1.3
- LED19 pad 1: +5V -> /rgb-led_matrix/C1.12
- LED19 pad 2: /switch_matrix/K_F10/DOUT -> /rgb-led_matrix/S1.1
- LED19 pad 3: GND -> /rgb-led_matrix/S1.2
- LED19 pad 4: /switch_matrix/K_F10/DIN -> /rgb-led_matrix/S1.3
- LED2 pad 1: +5V -> /rgb-led_matrix/C1.5
- LED2 pad 2: /switch_matrix/K_M2/DOUT -> /rgb-led_matrix/S1.1
- LED2 pad 3: GND -> /rgb-led_matrix/S1.2
- LED2 pad 4: /switch_matrix/K_M1/DOUT -> /rgb-led_matrix/S1.3
- LED20 pad 1: +5V -> /rgb-led_matrix/C2.1
- LED20 pad 2: /switch_matrix/K_F10/DIN -> /rgb-led_matrix/S2.1
- LED20 pad 3: GND -> /rgb-led_matrix/S2.2
- LED20 pad 4: /switch_matrix/K_F11/DIN -> /rgb-led_matrix/S2.3
- LED21 pad 1: +5V -> /rgb-led_matrix/C2.2
- LED21 pad 2: /switch_matrix/K_F11/DIN -> /rgb-led_matrix/S2.1
- LED21 pad 3: GND -> /rgb-led_matrix/S2.2
- LED21 pad 4: /switch_matrix/K_F12/DIN -> /rgb-led_matrix/S2.3
- LED22 pad 1: +5V -> /rgb-led_matrix/C2.3
- LED22 pad 2: /switch_matrix/K_F12/DIN -> /rgb-led_matrix/S2.1
- LED22 pad 3: GND -> /rgb-led_matrix/S2.2
- LED22 pad 4: /switch_matrix/K_PRTSC/DIN -> /rgb-led_matrix/S2.3
- LED23 pad 1: +5V -> /rgb-led_matrix/C2.3
- LED23 pad 2: /switch_matrix/K_PRTSC/DIN -> /rgb-led_matrix/S2.1
- LED23 pad 3: GND -> /rgb-led_matrix/S2.2
- LED23 pad 4: /switch_matrix/K_PAUSE/DOUT -> /rgb-led_matrix/S2.3
- LED24 pad 1: +5V -> /rgb-led_matrix/C2.4
- LED24 pad 2: /switch_matrix/K_PAUSE/DOUT -> /rgb-led_matrix/S2.1
- LED24 pad 3: GND -> /rgb-led_matrix/S2.2
- LED24 pad 4: /switch_matrix/K_PAUSE/DIN -> /rgb-led_matrix/S2.3
- LED25 pad 1: +5V -> /rgb-led_matrix/C2.5
- LED25 pad 2: /switch_matrix/K_PAUSE/DIN -> /rgb-led_matrix/S2.1
- LED25 pad 3: GND -> /rgb-led_matrix/S2.2
- LED25 pad 4: /switch_matrix/K_Play/DOUT -> /rgb-led_matrix/S2.3
- LED26 pad 1: +5V -> /rgb-led_matrix/C2.6
- LED26 pad 2: /switch_matrix/K_Play/DOUT -> /rgb-led_matrix/S2.1
- LED26 pad 3: GND -> /rgb-led_matrix/S2.2
- LED26 pad 4: /switch_matrix/K_Next/DOUT -> /rgb-led_matrix/S2.3
- LED27 pad 1: +5V -> /rgb-led_matrix/C2.7
- LED27 pad 2: /switch_matrix/K_Next/DOUT -> /rgb-led_matrix/S2.1
- LED27 pad 3: GND -> /rgb-led_matrix/S2.2
- LED27 pad 4: /switch_matrix/K_Mute/DOUT -> /rgb-led_matrix/S2.3
- LED28 pad 1: +5V -> /rgb-led_matrix/C2.8
- LED28 pad 2: /switch_matrix/K_Mute/DOUT -> /rgb-led_matrix/S2.1
- LED28 pad 3: GND -> /rgb-led_matrix/S2.2
- LED28 pad 4: /switch_matrix/K_Brightness/DOUT -> /rgb-led_matrix/S2.3
- LED29 pad 1: +5V -> /rgb-led_matrix/C2.9
- LED29 pad 2: /switch_matrix/K_G1/DOUT -> /rgb-led_matrix/S2.1
- LED29 pad 3: GND -> /rgb-led_matrix/S2.2
- LED29 pad 4: /switch_matrix/K_ESC/DOUT -> /rgb-led_matrix/S2.3
- LED3 pad 1: +5V -> /rgb-led_matrix/C1.6
- LED3 pad 2: /switch_matrix/K_M3/DOUT -> /rgb-led_matrix/S1.1
- LED3 pad 3: GND -> /rgb-led_matrix/S1.2
- LED3 pad 4: /switch_matrix/K_M2/DOUT -> /rgb-led_matrix/S1.3
- LED30 pad 1: +5V -> /rgb-led_matrix/C2.10
- LED30 pad 2: /switch_matrix/K_1/DIN -> /rgb-led_matrix/S2.1
- LED30 pad 3: GND -> /rgb-led_matrix/Mac\Win/GRN
- LED30 pad 4: /switch_matrix/K_G1/DOUT -> /rgb-led_matrix/Mac\Win/BLU
- LED31 pad 1: +5V -> /rgb-led_matrix/C1.2
- LED31 pad 2: /switch_matrix/K_1/DOUT -> /rgb-led_matrix/S1.4
- LED31 pad 3: GND -> /rgb-led_matrix/S1.5
- LED31 pad 4: /switch_matrix/K_1/DIN -> /rgb-led_matrix/S1.6
- LED32 pad 1: +5V -> /rgb-led_matrix/C1.3
- LED32 pad 2: /switch_matrix/K_2/DOUT -> /rgb-led_matrix/S1.4
- LED32 pad 3: GND -> /rgb-led_matrix/S1.5
- LED32 pad 4: /switch_matrix/K_1/DOUT -> /rgb-led_matrix/S1.6
- LED33 pad 1: +5V -> /rgb-led_matrix/C1.4
- LED33 pad 2: /switch_matrix/K_3/DOUT -> /rgb-led_matrix/S1.4
- LED33 pad 3: GND -> /rgb-led_matrix/S1.5
- LED33 pad 4: /switch_matrix/K_2/DOUT -> /rgb-led_matrix/S1.6
- LED34 pad 1: +5V -> /rgb-led_matrix/C1.5
- LED34 pad 2: /switch_matrix/K_4/DOUT -> /rgb-led_matrix/S1.4
- LED34 pad 3: GND -> /rgb-led_matrix/S1.5
- LED34 pad 4: /switch_matrix/K_3/DOUT -> /rgb-led_matrix/S1.6
- LED35 pad 1: +5V -> /rgb-led_matrix/C1.6
- LED35 pad 2: /switch_matrix/K_5/DOUT -> /rgb-led_matrix/S1.4
- LED35 pad 3: GND -> /rgb-led_matrix/S1.5
- LED35 pad 4: /switch_matrix/K_4/DOUT -> /rgb-led_matrix/S1.6
- LED36 pad 1: +5V -> /rgb-led_matrix/C1.7
- LED36 pad 2: /switch_matrix/K_6/DOUT -> /rgb-led_matrix/S1.4
- LED36 pad 3: GND -> /rgb-led_matrix/S1.5
- LED36 pad 4: /switch_matrix/K_5/DOUT -> /rgb-led_matrix/S1.6
- LED37 pad 1: +5V -> /rgb-led_matrix/C1.8
- LED37 pad 2: /switch_matrix/K_7/DOUT -> /rgb-led_matrix/S1.4
- LED37 pad 3: GND -> /rgb-led_matrix/S1.5
- LED37 pad 4: /switch_matrix/K_6/DOUT -> /rgb-led_matrix/S1.6
- LED38 pad 1: +5V -> /rgb-led_matrix/C1.9
- LED38 pad 2: /switch_matrix/K_8/DOUT -> /rgb-led_matrix/S1.4
- LED38 pad 3: GND -> /rgb-led_matrix/S1.5
- LED38 pad 4: /switch_matrix/K_7/DOUT -> /rgb-led_matrix/S1.6
- LED39 pad 1: +5V -> /rgb-led_matrix/C1.10
- LED39 pad 2: /switch_matrix/K_0/DIN -> /rgb-led_matrix/S1.4
- LED39 pad 3: GND -> /rgb-led_matrix/S1.5
- LED39 pad 4: /switch_matrix/K_8/DOUT -> /rgb-led_matrix/S1.6
- LED4 pad 1: +5V -> /rgb-led_matrix/C1.7
- LED4 pad 2: /switch_matrix/K_MR/DOUT -> /rgb-led_matrix/S1.1
- LED4 pad 3: GND -> /rgb-led_matrix/S1.2
- LED4 pad 4: /switch_matrix/K_M3/DOUT -> /rgb-led_matrix/S1.3
- LED40 pad 1: +5V -> /rgb-led_matrix/C1.11
- LED40 pad 2: /switch_matrix/K_0/DOUT -> /rgb-led_matrix/S1.4
- LED40 pad 3: GND -> /rgb-led_matrix/S1.5
- LED40 pad 4: /switch_matrix/K_0/DIN -> /rgb-led_matrix/S1.6
- LED41 pad 1: +5V -> /rgb-led_matrix/C1.12
- LED41 pad 2: /switch_matrix/K_Equals/DIN -> /rgb-led_matrix/S1.4
- LED41 pad 3: GND -> /rgb-led_matrix/S1.5
- LED41 pad 4: /switch_matrix/K_0/DOUT -> /rgb-led_matrix/S1.6
- LED42 pad 1: +5V -> /rgb-led_matrix/C2.1
- LED42 pad 2: /switch_matrix/K_Backspace/DIN -> /rgb-led_matrix/S2.4
- LED42 pad 3: GND -> /rgb-led_matrix/S2.5
- LED42 pad 4: /switch_matrix/K_Equals/DIN -> /rgb-led_matrix/S2.6
- LED43 pad 1: +5V -> /rgb-led_matrix/C2.2
- LED43 pad 2: /switch_matrix/K_Backspace/DOUT -> /rgb-led_matrix/S2.4
- LED43 pad 3: GND -> /rgb-led_matrix/S2.5
- LED43 pad 4: /switch_matrix/K_Backspace/DIN -> /rgb-led_matrix/S2.6
- LED44 pad 1: +5V -> /rgb-led_matrix/C2.3
- LED44 pad 2: /switch_matrix/K_HOME/DIN -> /rgb-led_matrix/S2.4
- LED44 pad 3: GND -> /rgb-led_matrix/S2.5
- LED44 pad 4: /switch_matrix/K_Backspace/DOUT -> /rgb-led_matrix/S2.6
- LED45 pad 1: +5V -> /rgb-led_matrix/C2.4
- LED45 pad 2: /switch_matrix/K_HOME/DOUT -> /rgb-led_matrix/S2.4
- LED45 pad 3: GND -> /rgb-led_matrix/S2.5
- LED45 pad 4: /switch_matrix/K_HOME/DIN -> /rgb-led_matrix/S2.6
- LED46 pad 1: +5V -> /rgb-led_matrix/C2.5
- LED46 pad 2: /switch_matrix/K_PGUP/DOUT -> /rgb-led_matrix/S2.4
- LED46 pad 3: GND -> /rgb-led_matrix/S2.5
- LED46 pad 4: /switch_matrix/K_HOME/DOUT -> /rgb-led_matrix/S2.6
- LED47 pad 1: +5V -> /rgb-led_matrix/C2.6
- LED47 pad 2: /switch_matrix/K_npNUM/DOUT -> /rgb-led_matrix/S2.4
- LED47 pad 3: GND -> /rgb-led_matrix/S2.5
- LED47 pad 4: /switch_matrix/K_PGUP/DOUT -> /rgb-led_matrix/S2.6
- LED48 pad 1: +5V -> /rgb-led_matrix/C2.7
- LED48 pad 2: /switch_matrix/K_npAsterisk/DIN -> /rgb-led_matrix/S2.4
- LED48 pad 3: GND -> /rgb-led_matrix/S2.5
- LED48 pad 4: /switch_matrix/K_npNUM/DOUT -> /rgb-led_matrix/S2.6
- LED49 pad 1: +5V -> /rgb-led_matrix/C2.8
- LED49 pad 2: /switch_matrix/K_npAsterisk/DOUT -> /rgb-led_matrix/S2.4
- LED49 pad 3: GND -> /rgb-led_matrix/S2.5
- LED49 pad 4: /switch_matrix/K_npAsterisk/DIN -> /rgb-led_matrix/S2.6
- LED5 pad 1: +5V -> /rgb-led_matrix/C1.7
- LED5 pad 2: /switch_matrix/K_Bluetooth/DIN -> /rgb-led_matrix/S1.1
- LED5 pad 3: GND -> /rgb-led_matrix/S1.2
- LED5 pad 4: /switch_matrix/K_MR/DOUT -> /rgb-led_matrix/S1.3
- LED50 pad 1: +5V -> /rgb-led_matrix/C2.9
- LED50 pad 2: /switch_matrix/K_np9/DIN -> /rgb-led_matrix/S2.4
- LED50 pad 3: GND -> /rgb-led_matrix/S2.5
- LED50 pad 4: /switch_matrix/K_npAsterisk/DOUT -> /rgb-led_matrix/S2.6
- LED51 pad 1: +5V -> /rgb-led_matrix/C2.10
- LED51 pad 2: /switch_matrix/K_G2/DOUT -> /rgb-led_matrix/S2.4
- LED51 pad 3: GND -> /rgb-led_matrix/S2.5
- LED51 pad 4: /switch_matrix/K_G2/DIN -> /rgb-led_matrix/S2.6
- LED52 pad 1: +5V -> /rgb-led_matrix/C1.2
- LED52 pad 2: /switch_matrix/K_G2/DIN -> /rgb-led_matrix/S1.4
- LED52 pad 3: GND -> /rgb-led_matrix/S1.5
- LED52 pad 4: /switch_matrix/K_Q/DOUT -> /rgb-led_matrix/S1.6
- LED53 pad 1: +5V -> /rgb-led_matrix/C1.3
- LED53 pad 2: /switch_matrix/K_Q/DOUT -> /rgb-led_matrix/S1.4
- LED53 pad 3: GND -> /rgb-led_matrix/S1.5
- LED53 pad 4: /switch_matrix/K_Q/DIN -> /rgb-led_matrix/S1.6
- LED54 pad 1: +5V -> /rgb-led_matrix/C1.4
- LED54 pad 2: /switch_matrix/K_Q/DIN -> /rgb-led_matrix/S1.4
- LED54 pad 3: GND -> /rgb-led_matrix/S1.5
- LED54 pad 4: /switch_matrix/K_E/DOUT -> /rgb-led_matrix/S1.6
- LED55 pad 1: +5V -> /rgb-led_matrix/C1.5
- LED55 pad 2: /switch_matrix/K_E/DOUT -> /rgb-led_matrix/S1.4
- LED55 pad 3: GND -> /rgb-led_matrix/S1.5
- LED55 pad 4: /switch_matrix/K_E/DIN -> /rgb-led_matrix/S1.6
- LED56 pad 1: +5V -> /rgb-led_matrix/C1.6
- LED56 pad 2: /switch_matrix/K_E/DIN -> /rgb-led_matrix/S1.4
- LED56 pad 3: GND -> /rgb-led_matrix/S1.5
- LED56 pad 4: /switch_matrix/K_R/DIN -> /rgb-led_matrix/S1.6
- LED57 pad 1: +5V -> /rgb-led_matrix/C1.7
- LED57 pad 2: /switch_matrix/K_R/DIN -> /rgb-led_matrix/S1.4
- LED57 pad 3: GND -> /rgb-led_matrix/S1.5
- LED57 pad 4: /switch_matrix/K_T/DIN -> /rgb-led_matrix/S1.6
- LED58 pad 1: +5V -> /rgb-led_matrix/C1.8
- LED58 pad 2: /switch_matrix/K_T/DIN -> /rgb-led_matrix/S1.4
- LED58 pad 3: GND -> /rgb-led_matrix/S1.5
- LED58 pad 4: /switch_matrix/K_U/DOUT -> /rgb-led_matrix/S1.6
- LED59 pad 1: +5V -> /rgb-led_matrix/C1.9
- LED59 pad 2: /switch_matrix/K_U/DOUT -> /rgb-led_matrix/S1.4
- LED59 pad 3: GND -> /rgb-led_matrix/S1.5
- LED59 pad 4: /switch_matrix/K_I/DOUT -> /rgb-led_matrix/S1.6
- LED6 pad 1: +5V -> /rgb-led_matrix/C1.7
- LED6 pad 2: /switch_matrix/K_Bluetooth/DOUT -> /rgb-led_matrix/S1.1
- LED6 pad 3: GND -> /rgb-led_matrix/S1.2
- LED6 pad 4: /switch_matrix/K_Bluetooth/DIN -> /rgb-led_matrix/S1.3
- LED60 pad 1: +5V -> /rgb-led_matrix/C1.10
- LED60 pad 2: /switch_matrix/K_I/DOUT -> /rgb-led_matrix/S1.4
- LED60 pad 3: GND -> /rgb-led_matrix/S1.5
- LED60 pad 4: /switch_matrix/K_I/DIN -> /rgb-led_matrix/S1.6
- LED61 pad 1: +5V -> /rgb-led_matrix/C1.11
- LED61 pad 2: /switch_matrix/K_I/DIN -> /rgb-led_matrix/S1.4
- LED61 pad 3: GND -> /rgb-led_matrix/S1.5
- LED61 pad 4: /switch_matrix/K_O/DIN -> /rgb-led_matrix/S1.6
- LED62 pad 1: +5V -> /rgb-led_matrix/C1.12
- LED62 pad 2: /switch_matrix/K_O/DIN -> /rgb-led_matrix/S1.4
- LED62 pad 3: GND -> /rgb-led_matrix/S1.5
- LED62 pad 4: /switch_matrix/K_LBracket/DOUT -> /rgb-led_matrix/S1.6
- LED63 pad 1: +5V -> /rgb-led_matrix/C2.1
- LED63 pad 2: /switch_matrix/K_LBracket/DOUT -> /rgb-led_matrix/S2.4
- LED63 pad 3: GND -> /rgb-led_matrix/S2.5
- LED63 pad 4: /switch_matrix/K_LBracket/DIN -> /rgb-led_matrix/S2.6
- LED64 pad 1: +5V -> /rgb-led_matrix/C2.2
- LED64 pad 2: /switch_matrix/K_LBracket/DIN -> /rgb-led_matrix/S2.4
- LED64 pad 3: GND -> /rgb-led_matrix/S2.5
- LED64 pad 4: /switch_matrix/K_Backslash/DOUT -> /rgb-led_matrix/S2.6
- LED65 pad 1: +5V -> /rgb-led_matrix/C2.3
- LED65 pad 2: /switch_matrix/K_Backslash/DOUT -> /rgb-led_matrix/S2.4
- LED65 pad 3: GND -> /rgb-led_matrix/S2.5
- LED65 pad 4: /switch_matrix/K_Backslash/DIN -> /rgb-led_matrix/S2.6
- LED66 pad 1: +5V -> /rgb-led_matrix/C2.4
- LED66 pad 2: /switch_matrix/K_Backslash/DIN -> /rgb-led_matrix/S2.4
- LED66 pad 3: GND -> /rgb-led_matrix/S2.5
- LED66 pad 4: /switch_matrix/K_DEL/DIN -> /rgb-led_matrix/S2.6
- LED67 pad 1: +5V -> /rgb-led_matrix/C2.5
- LED67 pad 2: /switch_matrix/K_DEL/DIN -> /rgb-led_matrix/S2.4
- LED67 pad 3: GND -> /rgb-led_matrix/S2.5
- LED67 pad 4: /switch_matrix/K_END/DIN -> /rgb-led_matrix/S2.6
- LED68 pad 1: +5V -> /rgb-led_matrix/C2.6
- LED68 pad 2: /switch_matrix/K_END/DIN -> /rgb-led_matrix/S2.4
- LED68 pad 3: GND -> /rgb-led_matrix/S2.5
- LED68 pad 4: /switch_matrix/K_PGDN/DIN -> /rgb-led_matrix/S2.6
- LED69 pad 1: +5V -> /rgb-led_matrix/C2.7
- LED69 pad 2: /switch_matrix/K_PGDN/DIN -> /rgb-led_matrix/S2.4
- LED69 pad 3: GND -> /rgb-led_matrix/S2.5
- LED69 pad 4: /switch_matrix/K_np7/DIN -> /rgb-led_matrix/S2.6
- LED7 pad 1: +5V -> /rgb-led_matrix/C1.9
- LED7 pad 2: /switch_matrix/K_Brightness/DIN -> /rgb-led_matrix/S1.1
- LED7 pad 3: GND -> /rgb-led_matrix/S1.2
- LED7 pad 4: /switch_matrix/K_Bluetooth/DOUT -> /rgb-led_matrix/S1.3
- LED70 pad 1: +5V -> /rgb-led_matrix/C2.8
- LED70 pad 2: /switch_matrix/K_np7/DIN -> /rgb-led_matrix/S2.4
- LED70 pad 3: GND -> /rgb-led_matrix/S2.5
- LED70 pad 4: /switch_matrix/K_np8/DIN -> /rgb-led_matrix/S2.6
- LED71 pad 1: +5V -> /rgb-led_matrix/C2.9
- LED71 pad 2: /switch_matrix/K_np8/DIN -> /rgb-led_matrix/S2.4
- LED71 pad 3: GND -> /rgb-led_matrix/S2.5
- LED71 pad 4: /switch_matrix/K_np9/DIN -> /rgb-led_matrix/S2.6
- LED72 pad 1: +5V -> /rgb-led_matrix/C1.2
- LED72 pad 2: /switch_matrix/K_np3/DIN -> /rgb-led_matrix/S1.7
- LED72 pad 3: GND -> /rgb-led_matrix/S1.8
- LED72 pad 4: /switch_matrix/K_np6/DOUT -> /rgb-led_matrix/S1.9
- LED73 pad 1: +5V -> /rgb-led_matrix/C1.3
- LED73 pad 2: /switch_matrix/K_CAPS/DIN -> /rgb-led_matrix/S1.7
- LED73 pad 3: GND -> /rgb-led_matrix/S1.8
- LED73 pad 4: /switch_matrix/K_G2/DOUT -> /rgb-led_matrix/S1.9
- LED74 pad 1: +5V -> /rgb-led_matrix/C1.4
- LED74 pad 2: /switch_matrix/K_A/DIN -> /rgb-led_matrix/S1.7
- LED74 pad 3: GND -> /rgb-led_matrix/S1.8
- LED74 pad 4: /switch_matrix/K_CAPS/DIN -> /rgb-led_matrix/S1.9
- LED75 pad 1: +5V -> /rgb-led_matrix/C1.5
- LED75 pad 2: /switch_matrix/K_A/DOUT -> /rgb-led_matrix/S1.7
- LED75 pad 3: GND -> /rgb-led_matrix/S1.8
- LED75 pad 4: /switch_matrix/K_A/DIN -> /rgb-led_matrix/S1.9
- LED76 pad 1: +5V -> /rgb-led_matrix/C1.6
- LED76 pad 2: /switch_matrix/K_D/DIN -> /rgb-led_matrix/S1.7
- LED76 pad 3: GND -> /rgb-led_matrix/S1.8
- LED76 pad 4: /switch_matrix/K_A/DOUT -> /rgb-led_matrix/S1.9
- LED77 pad 1: +5V -> /rgb-led_matrix/C1.7
- LED77 pad 2: /switch_matrix/K_D/DOUT -> /rgb-led_matrix/S1.7
- LED77 pad 3: GND -> /rgb-led_matrix/S1.8
- LED77 pad 4: /switch_matrix/K_D/DIN -> /rgb-led_matrix/S1.9
- LED78 pad 1: +5V -> /rgb-led_matrix/C1.8
- LED78 pad 2: /switch_matrix/K_F/DOUT -> /rgb-led_matrix/S1.7
- LED78 pad 3: GND -> /rgb-led_matrix/S1.8
- LED78 pad 4: /switch_matrix/K_D/DOUT -> /rgb-led_matrix/S1.9
- LED79 pad 1: +5V -> /rgb-led_matrix/C1.9
- LED79 pad 2: /switch_matrix/K_G/DOUT -> /rgb-led_matrix/S1.7
- LED79 pad 3: GND -> /rgb-led_matrix/S1.8
- LED79 pad 4: /switch_matrix/K_F/DOUT -> /rgb-led_matrix/S1.9
- LED8 pad 1: +5V -> /rgb-led_matrix/C1.10
- LED8 pad 2: /switch_matrix/K_Brightness/DOUT -> /rgb-led_matrix/S1.1
- LED8 pad 3: GND -> /rgb-led_matrix/S1.2
- LED8 pad 4: /switch_matrix/K_Brightness/DIN -> /rgb-led_matrix/S1.3
- LED80 pad 1: +5V -> /rgb-led_matrix/C1.10
- LED80 pad 2: /switch_matrix/K_H/DOUT -> /rgb-led_matrix/S1.7
- LED80 pad 3: GND -> /rgb-led_matrix/S1.8
- LED80 pad 4: /switch_matrix/K_G/DOUT -> /rgb-led_matrix/S1.9
- LED81 pad 1: +5V -> /rgb-led_matrix/C1.11
- LED81 pad 2: /switch_matrix/K_J/DOUT -> /rgb-led_matrix/S1.7
- LED81 pad 3: GND -> /rgb-led_matrix/S1.8
- LED81 pad 4: /switch_matrix/K_H/DOUT -> /rgb-led_matrix/S1.9
- LED82 pad 1: +5V -> /rgb-led_matrix/C1.12
- LED82 pad 2: /switch_matrix/K_K/DOUT -> /rgb-led_matrix/S1.7
- LED82 pad 3: GND -> /rgb-led_matrix/S1.8
- LED82 pad 4: /switch_matrix/K_J/DOUT -> /rgb-led_matrix/S1.9
- LED83 pad 1: +5V -> /rgb-led_matrix/C2.1
- LED83 pad 2: /switch_matrix/K_L/DOUT -> /rgb-led_matrix/S2.7
- LED83 pad 3: GND -> /rgb-led_matrix/S2.8
- LED83 pad 4: /switch_matrix/K_K/DOUT -> /rgb-led_matrix/S2.9
- LED84 pad 1: +5V -> /rgb-led_matrix/C2.2
- LED84 pad 2: /switch_matrix/K_Apostrophe/DIN -> /rgb-led_matrix/S2.7
- LED84 pad 3: GND -> /rgb-led_matrix/S2.8
- LED84 pad 4: /switch_matrix/K_L/DOUT -> /rgb-led_matrix/S2.9
- LED85 pad 1: +5V -> /rgb-led_matrix/C2.7
- LED85 pad 2: /switch_matrix/K_Apostrophe/DOUT -> /rgb-led_matrix/S2.7
- LED85 pad 3: GND -> /rgb-led_matrix/S2.8
- LED85 pad 4: /switch_matrix/K_Apostrophe/DIN -> /rgb-led_matrix/S2.9
- LED86 pad 1: +5V -> /rgb-led_matrix/C2.8
- LED86 pad 2: /switch_matrix/K_ENTER/DOUT -> /rgb-led_matrix/S2.7
- LED86 pad 3: GND -> /rgb-led_matrix/S2.8
- LED86 pad 4: /switch_matrix/K_Apostrophe/DOUT -> /rgb-led_matrix/S2.9
- LED87 pad 1: +5V -> /rgb-led_matrix/C2.9
- LED87 pad 2: /switch_matrix/K_np4/DOUT -> /rgb-led_matrix/S2.7
- LED87 pad 3: GND -> /rgb-led_matrix/S2.8
- LED87 pad 4: /switch_matrix/K_ENTER/DOUT -> /rgb-led_matrix/S2.9
- LED88 pad 1: +5V -> /rgb-led_matrix/C1.2
- LED88 pad 2: /switch_matrix/K_np5/DOUT -> /rgb-led_matrix/S1.7
- LED88 pad 3: GND -> /rgb-led_matrix/S1.8
- LED88 pad 4: /switch_matrix/K_np4/DOUT -> /rgb-led_matrix/S1.9
- LED89 pad 1: +5V -> /rgb-led_matrix/C1.3
- LED89 pad 2: /switch_matrix/K_np6/DOUT -> /rgb-led_matrix/S1.7
- LED89 pad 3: GND -> /rgb-led_matrix/S1.8
- LED89 pad 4: /switch_matrix/K_np5/DOUT -> /rgb-led_matrix/S1.9
- LED9 pad 1: +5V -> /rgb-led_matrix/C1.11
- LED9 pad 2: /switch_matrix/K_ESC/DOUT -> /rgb-led_matrix/S1.1
- LED9 pad 3: GND -> /rgb-led_matrix/S1.2
- LED9 pad 4: /switch_matrix/K_ESC/DIN -> /rgb-led_matrix/S1.3
- LED90 pad 1: +5V -> /rgb-led_matrix/X/AN
- LED90 pad 2: /switch_matrix/K_G4/DOUT -> /rgb-led_matrix/S1.7
- LED90 pad 3: GND -> /rgb-led_matrix/S1.8
- LED90 pad 4: /switch_matrix/K_G4/DIN -> /rgb-led_matrix/S1.9
- LED91 pad 1: +5V -> /rgb-led_matrix/C1.5
- LED91 pad 2: /switch_matrix/K_G4/DIN -> /rgb-led_matrix/S1.7
- LED91 pad 3: GND -> /rgb-led_matrix/S1.8
- LED91 pad 4: /switch_matrix/K_LSHIFT/DIN -> /rgb-led_matrix/S1.9
- LED92 pad 1: +5V -> /rgb-led_matrix/C1.6
- LED92 pad 2: /switch_matrix/K_LSHIFT/DIN -> /rgb-led_matrix/S1.7
- LED92 pad 3: GND -> /rgb-led_matrix/S1.8
- LED92 pad 4: /switch_matrix/K_X/DOUT -> /rgb-led_matrix/S1.9
- LED93 pad 1: +5V -> /rgb-led_matrix/C1.7
- LED93 pad 2: /switch_matrix/K_X/DOUT -> /rgb-led_matrix/S1.7
- LED93 pad 3: GND -> /rgb-led_matrix/S1.8
- LED93 pad 4: /switch_matrix/K_C/DOUT -> /rgb-led_matrix/S1.9
- LED94 pad 1: +5V -> /rgb-led_matrix/C1.8
- LED94 pad 2: /switch_matrix/K_C/DOUT -> /rgb-led_matrix/S1.7
- LED94 pad 3: GND -> /rgb-led_matrix/S1.8
- LED94 pad 4: /switch_matrix/K_C/DIN -> /rgb-led_matrix/S1.9
- LED95 pad 1: +5V -> /rgb-led_matrix/C1.9
- LED95 pad 2: /switch_matrix/K_C/DIN -> /rgb-led_matrix/S1.7
- LED95 pad 3: GND -> /rgb-led_matrix/S1.8
- LED95 pad 4: /switch_matrix/K_B/DOUT -> /rgb-led_matrix/S1.9
- LED96 pad 1: +5V -> /rgb-led_matrix/C1.10
- LED96 pad 2: /switch_matrix/K_B/DOUT -> /rgb-led_matrix/S1.7
- LED96 pad 3: GND -> /rgb-led_matrix/S1.8
- LED96 pad 4: /switch_matrix/K_B/DIN -> /rgb-led_matrix/S1.9
- LED97 pad 1: +5V -> /rgb-led_matrix/C1.11
- LED97 pad 2: /switch_matrix/K_B/DIN -> /rgb-led_matrix/S1.7
- LED97 pad 3: GND -> /rgb-led_matrix/S1.8
- LED97 pad 4: /switch_matrix/K_M/DOUT -> /rgb-led_matrix/S1.9
- LED98 pad 1: +5V -> /rgb-led_matrix/C1.12
- LED98 pad 2: /switch_matrix/K_M/DOUT -> /rgb-led_matrix/S1.7
- LED98 pad 3: GND -> /rgb-led_matrix/S1.8
- LED98 pad 4: /switch_matrix/K_Comma/DOUT -> /rgb-led_matrix/S1.9
- LED99 pad 1: +5V -> /rgb-led_matrix/C2.2
- LED99 pad 2: /switch_matrix/K_Comma/DOUT -> /rgb-led_matrix/S2.7
- LED99 pad 3: GND -> /rgb-led_matrix/S2.8
- LED99 pad 4: /switch_matrix/K_Comma/DIN -> /rgb-led_matrix/S2.9
- MX100 pad 2: /COL9 -> /switch_matrix/COL13
- MX101 pad 2: /COL10 -> /switch_matrix/COL16
- MX102 pad 2: /COL13 -> /switch_matrix/COL18
- MX103 pad 2: /COL15 -> /switch_matrix/COL19
- MX104 pad 2: /COL17 -> /switch_matrix/COL20
- MX105 pad 2: /COL18 -> /switch_matrix/COL21
- MX106 pad 2: /COL19 -> /switch_matrix/COL1
- MX107 pad 2: /COL20 -> /switch_matrix/COL1
- MX108 pad 2: /COLM -> /switch_matrix/COL2
- MX109 pad 2: /COL0 -> /switch_matrix/COL6
- MX11 pad 2: /COL3 -> /switch_matrix/COL1
- MX110 pad 2: /COL1 -> /switch_matrix/COL9
- MX111 pad 2: /COL2 -> /switch_matrix/COL10
- MX112 pad 2: /COL5 -> /switch_matrix/COL12
- MX113 pad 2: /COL8 -> /switch_matrix/COL13
- MX114 pad 2: /COL9 -> /switch_matrix/COL15
- MX115 pad 2: /COL11 -> /switch_matrix/COL16
- MX116 pad 2: /COL13 -> /switch_matrix/COL17
- MX117 pad 2: /COL14 -> /switch_matrix/COL18
- MX118 pad 2: /COL15 -> /switch_matrix/COL20
- MX12 pad 2: /COL4 -> /switch_matrix/COL3
- MX13 pad 2: /COL5 -> /switch_matrix/COL4
- MX14 pad 2: /COL6 -> /switch_matrix/COL8
- MX15 pad 2: /COL7 -> /switch_matrix/COL5
- MX16 pad 2: /COL8 -> /switch_matrix/COL6
- MX17 pad 2: /COL9 -> /switch_matrix/COL9
- MX18 pad 2: /COL11 -> /switch_matrix/COL10
- MX19 pad 2: /COL12 -> /switch_matrix/COL11
- MX20 pad 2: /COL13 -> /switch_matrix/COL12
- MX21 pad 2: /COL14 -> /switch_matrix/COL13
- MX22 pad 2: /COL14 -> /switch_matrix/COL14
- MX23 pad 2: /COL15 -> /switch_matrix/COL14
- MX24 pad 2: /COL16 -> /switch_matrix/COL15
- MX31 pad 2: /COL1 -> /switch_matrix/COL1
- MX32 pad 2: /COL2 -> /switch_matrix/COL2
- MX33 pad 2: /COL3 -> /switch_matrix/COL3
- MX34 pad 2: /COL4 -> /switch_matrix/COL4
- MX35 pad 2: /COL5 -> /switch_matrix/COL5
- MX36 pad 2: /COL6 -> /switch_matrix/COL6
- MX37 pad 2: /COL7 -> /switch_matrix/COL7
- MX38 pad 2: /COL8 -> /switch_matrix/COL8
- MX39 pad 2: /COL9 -> /switch_matrix/COL9
- MX40 pad 2: /COL10 -> /switch_matrix/COL10
- MX41 pad 2: /COL11 -> /switch_matrix/COL11
- MX42 pad 2: /COL12 -> /switch_matrix/COL12
- MX43 pad 2: /COL13 -> /switch_matrix/COL13
- MX44 pad 2: /COL14 -> /switch_matrix/COL14
- MX45 pad 2: /COL15 -> /switch_matrix/COL15
- MX46 pad 2: /COL16 -> /switch_matrix/COL16
- MX47 pad 2: /COL17 -> /switch_matrix/COL17
- MX48 pad 2: /COL18 -> /switch_matrix/COL18
- MX49 pad 2: /COL19 -> /switch_matrix/COL19
- MX50 pad 2: /COL20 -> /switch_matrix/COL20
- MX51 pad 2: /COLM -> /switch_matrix/COL21
- MX52 pad 2: /COL0 -> /switch_matrix/COL1
- MX53 pad 2: /COL1 -> /switch_matrix/COL2
- MX54 pad 2: /COL2 -> /switch_matrix/COL3
- MX55 pad 2: /COL3 -> /switch_matrix/COL4
- MX56 pad 2: /COL4 -> /switch_matrix/COL5
- MX57 pad 2: /COL5 -> /switch_matrix/COL6
- MX58 pad 2: /COL6 -> /switch_matrix/COL7
- MX59 pad 2: /COL7 -> /switch_matrix/COL8
- MX60 pad 2: /COL8 -> /switch_matrix/COL9
- MX61 pad 2: /COL9 -> /switch_matrix/COL10
- MX62 pad 2: /COL10 -> /switch_matrix/COL11
- MX63 pad 2: /COL11 -> /switch_matrix/COL12
- MX64 pad 2: /COL12 -> /switch_matrix/COL13
- MX65 pad 2: /COL13 -> /switch_matrix/COL14
- MX66 pad 2: /COL14 -> /switch_matrix/COL15
- MX67 pad 2: /COL15 -> /switch_matrix/COL16
- MX68 pad 2: /COL16 -> /switch_matrix/COL17
- MX69 pad 2: /COL17 -> /switch_matrix/COL18
- MX70 pad 2: /COL18 -> /switch_matrix/COL19
- MX71 pad 2: /COL19 -> /switch_matrix/COL20
- MX72 pad 2: /COL20 -> /switch_matrix/COL21
- MX73 pad 2: /COLM -> /switch_matrix/COL1
- MX74 pad 2: /COL0 -> /switch_matrix/COL2
- MX75 pad 2: /COL1 -> /switch_matrix/COL3
- MX76 pad 2: /COL2 -> /switch_matrix/COL4
- MX77 pad 2: /COL3 -> /switch_matrix/COL5
- MX78 pad 2: /COL4 -> /switch_matrix/COL6
- MX79 pad 2: /COL5 -> /switch_matrix/COL7
- MX80 pad 2: /COL6 -> /switch_matrix/COL8
- MX81 pad 2: /COL7 -> /switch_matrix/COL9
- MX82 pad 2: /COL8 -> /switch_matrix/COL10
- MX83 pad 2: /COL9 -> /switch_matrix/COL11
- MX84 pad 2: /COL10 -> /switch_matrix/COL12
- MX85 pad 2: /COL11 -> /switch_matrix/COL13
- MX86 pad 2: /COL13 -> /switch_matrix/COL18
- MX87 pad 2: /COL17 -> /switch_matrix/COL19
- MX88 pad 2: /COL18 -> /switch_matrix/COL20
- MX89 pad 2: /COL19 -> /switch_matrix/COL1
- MX90 pad 2: /COLM -> /switch_matrix/COL2
- MX91 pad 2: /COL0 -> /switch_matrix/COL3
- MX92 pad 2: /COL1 -> /switch_matrix/COL4
- MX93 pad 2: /COL2 -> /switch_matrix/COL5
- MX94 pad 2: /COL3 -> /switch_matrix/COL6
- MX95 pad 2: /COL4 -> /switch_matrix/COL7
- MX96 pad 2: /COL5 -> /switch_matrix/COL8
- MX97 pad 2: /COL6 -> /switch_matrix/COL9
- MX98 pad 2: /COL7 -> /switch_matrix/COL10
- MX99 pad 2: /COL8 -> /switch_matrix/COL11
- R10 pad 1: Net-(J4-CC2) -> Net-(Q1-PadG)
- R11 pad 1: GND -> Net-(J4-CC1)
- R11 pad 2: Net-(U4-ILIM) -> GND
- R12 pad 1: GND -> Net-(J4-CC2)
- R12 pad 2: Net-(U4-ISET) -> GND
- R13 pad 1: Net-(U4-ITERM) -> Net-(U3-TS)
- R14 pad 1: /VDDH -> GND
- R14 pad 2: Net-(D122-A) -> Net-(U3-ILIM)
- R15 pad 1: Net-(Q1-PadG) -> GND
- R15 pad 2: GND -> Net-(U3-ISET)
- R16 pad 1: /VBATT_nRF -> Net-(U3-ITERM)
- R16 pad 2: /USB and Power management/V_BATT -> GND
- R17 pad 1: GND -> /VDDH
- R17 pad 2: /VBATT_nRF -> Net-(D120-A)
- R18 pad 1: +5V -> /VBATT_nRF
- R18 pad 2: /~{RGB_EN} -> /USB and Power management/V_BATT
- R19 pad 1: Net-(D124-A) -> GND
- R19 pad 2: +5V -> /VBATT_nRF
- R21 pad 1: Net-(Q1-PadG) -> Net-(Q2-PadG)
- R22 pad 1: Net-(D123-A) -> Net-(Q2-PadG)
- R22 pad 2: +5V -> GND
- R8 pad 1: Net-(R8-Pad1) -> Net-(D119-A)
- R8 pad 2: /RGB_DIN -> +5V
- R9 pad 1: Net-(J4-CC1) -> Net-(Q1-PadG)
- R9 pad 2: GND -> /CAPS_LED
- TP1 pad 1: /switch_matrix/RGB_DOUT -> /RGB_DOUT
- U1 pad B13: /MCU_RGB -> /CAPS_LED
- U1 pad B19: /CAPS_LED -> unconnected-(U1-P1.11-PadB19)
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Routing:
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Other:
- outline, holes or cut-outs redrawn

Commit message: k618 pcb work
Parts:
- added REF**: stabilizer-cutout, K618:stabilizer-cutout, F.Cu at (493.9, 328.8)
- moved MX1 161.3 mm to (71.0, 80.8)
- moved MX10 161.3 mm to (366.6, 80.8)
- moved MX100 161.3 mm to (301.9, 178.7)
- moved MX101 161.3 mm to (361.7, 178.7)
- moved MX102 161.3 mm to (404.8, 178.7)
- moved MX103 161.3 mm to (423.8, 178.7)
- moved MX104 161.3 mm to (442.8, 178.7)
- moved MX105 161.3 mm to (461.8, 188.2)
- moved MX106 161.3 mm to (54.9, 197.7)
- moved MX107 161.3 mm to (78.7, 197.7)
- moved MX108 161.3 mm to (102.4, 197.7)
- moved MX109 161.3 mm to (173.7, 197.7)
- moved MX11 161.3 mm to (52.5, 99.8)
- moved MX110 161.3 mm to (244.9, 197.7)
- moved MX111 161.3 mm to (268.6, 197.7)
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Other:
- board size 431.9 x 138.7 mm -> 431.9 x 148.3 mm
- board text added: "15.5 (7.75)"
- board text added: "7.5 (3.75)"
