File: redragon-k618-pro/zmk-k618.kicad_pcb (KiCad board)
At the start: 2 copper layers, 431.9 x 148.3 mm, 591 parts, among them J1 Prog_conn, J2 Tag connect TC2030-CTX, J3 53047-0460, J4 TYPE-C-31-M12_13, J5 JST-4-pin, Q1 Q_NMOS, Q3 Q_NMOS, SW1 Reset Switch, U1 nRF52840-QIAA-R/nRF52833-QIAA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, U2 TPD4E05U06DQAR, U3 BQ24074RGTR, U4 BQ24074RGTR, Y1 32.768kHz, Y2 32MHz

Commit message: g915 and k618 pcb key and cutout placement
Parts:
- MX100, MX101, MX102, MX103, MX104, MX105, MX106, MX107, MX108, MX109, MX11, MX110, MX111, MX112, MX113, MX114, MX115, MX116, MX117, MX118, MX12, MX13, MX14, MX15, MX16, MX17, MX18, MX19, MX20, MX21, MX22, MX23, MX24, MX25, MX26, MX31, MX32, MX33, MX34, MX35, MX36, MX37, MX38, MX39, MX40, MX41, MX42, MX43, MX44, MX45, MX46, MX47, MX48, MX49, MX50, MX51, MX52, MX53, MX54, MX55, MX56, MX57, MX58, MX59, MX60, MX61, MX62, MX63, MX64, MX65, MX66, MX67, MX68, MX69, MX70, MX71, MX72, MX73, MX74, MX75, MX76, MX77, MX78, MX79, MX80, MX81, MX82, MX83, MX84, MX85, MX86, MX87, MX88, MX89, MX90, MX91, MX92, MX93, MX94, MX95, MX96, MX97, MX98, MX99: footprint key-switches:SW_Gateron_LowProfile_HotSwap_PTH -> key-switches:SW_Kailh_Choc_V1_THT
- moved REF** 502.0 mm to (-164.9, 290.4)
- moved REF** 502.0 mm to (-182.9, 290.4)
- moved REF** 502.0 mm to (-372.1, 290.4)
- moved REF** 502.0 mm to (-444.1, 290.4)
- moved REF** 502.0 mm to (-426.1, 290.4)
- moved REF** 502.0 mm to (-54.9, 311.3)
- moved REF** 502.0 mm to (-146.9, 290.4)
- moved REF** 502.0 mm to (-72.9, 311.3)
- moved REF** 502.0 mm to (-408.1, 290.4)
- moved REF** 502.0 mm to (-390.1, 290.4)
- moved REF** 502.0 mm to (-218.9, 290.4)
- moved REF** 502.0 mm to (-90.9, 311.3)
- moved REF** 502.0 mm to (-200.9, 290.4)
- moved REF** 502.0 mm to (-108.9, 311.3)
- moved MX24 163.4 mm to (326.8, 262.4)
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Other:
- board size 431.9 x 148.3 mm -> 431.9 x 138.7 mm
