File: redragon-k618-pro/key.kicad_sch (KiCad schematic)
At the start: 2 parts

Commit message: g915 and k618 pcb key and cutout placement
Parts:
- MX11: footprint key-switches:SW_Gateron_LowProfile_HotSwap_PTH -> key-switches:SW_Kailh_Choc_V1_THT
Changed lines of the file:
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@@
 			)
 		)
-		(property "Footprint" "key-switches:SW_Gateron_LowProfile_HotSwap_PTH"
+		(property "Footprint" "key-switches:SW_Kailh_Choc_V1_THT"
 			(at 144.78 114.3 0)
 			(effects
