File: dev-board/switch_matrix.kicad_sch (KiCad schematic)
At the start: 0 parts

Commit message: created dev-board to prove design before full-size
Other:
- removed sheet 0
- removed sheet 1
- removed sheet 2
- removed sheet 3
- removed sheet 4
- removed sheet 5
- removed sheet 6
- removed sheet 7
- removed sheet 8
- removed sheet 9
- removed sheet A
- removed sheet Apostrophe
- removed sheet B
- removed sheet Backslash
- removed sheet Backspace
- removed sheet Bluetooth
- removed sheet Brightness
- removed sheet C
- removed sheet CAPS
- removed sheet Comma
- removed sheet D
- removed sheet DEL
- removed sheet Dash
- removed sheet Down
- removed sheet E
- removed sheet END
- removed sheet ENTER
- removed sheet ESC
- removed sheet Equals
- removed sheet F
- removed sheet F1
- removed sheet F10
- removed sheet F11
- removed sheet F12
- removed sheet F2
- removed sheet F3
- removed sheet F4
- removed sheet F5
- removed sheet F6
- removed sheet F7
- removed sheet F8
- removed sheet F9
- removed sheet G
- removed sheet G1
- removed sheet G2
- removed sheet G3
- removed sheet G4
- removed sheet G5
- removed sheet GameMode
- removed sheet H
- removed sheet HOME
- removed sheet I
- removed sheet INS
- removed sheet J
- removed sheet K
- removed sheet L
- removed sheet LBracket
- removed sheet Left
- removed sheet M
- removed sheet M1
- removed sheet M2
- removed sheet M3
- removed sheet MR
- removed sheet Menu
- removed sheet N
- removed sheet O
- removed sheet P
- removed sheet PAUSE
- removed sheet PGDN
- removed sheet PGUP
- removed sheet PRTSC
- removed sheet Period
- removed sheet Q
- removed sheet R
- removed sheet RBracket
- removed sheet Right
- removed sheet S
- removed sheet SCRLK
- removed sheet Semicolon
- removed sheet Slash
- removed sheet Space
- removed sheet T
- removed sheet TAB
- removed sheet Tilde
- removed sheet U
- removed sheet Up
- removed sheet V
- removed sheet W
- removed sheet Wireless
- removed sheet X
- removed sheet Y
- removed sheet Z
- removed sheet lALT
- removed sheet lCTRL
- removed sheet lSHIFT
- removed sheet lWIN
- removed sheet rALT
- removed sheet rCTRL
- removed sheet rSHIFT
- removed sheet rWIN
- note added: "NOTE: Key instance sheet numbers (see 'Schematic Hierarchy' tree. ctrl+H if not visible) are used to ensure keys and associated components are annotated in an order that is compatible with kbplacer. This hack was needed becuase kbplacer uses ref des's to determine which components go where. Re-numbering the instance sheets was the easiest way to get it all to work together with the least amount o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"
- note removed: "NOTE: Key instance sheet numbers (see 'Schematic Hierarchy' tree. ctrl+H if not visible) are used to ensures keys and associated components are annotated in an order that is compatible with kbplacer. This hack was needed becuase kbplacer uses ref des's to determine which components go where. Re-numbering the instance sheets was the easiest way to get it all to work together with the least amount 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"
