File: dev-board/rgb-led_matrix.kicad_sch (KiCad schematic)
At the start: 21 parts, among them U4 IS31FL3733-TQ, U5 IS31FL3733-TQ

Commit message: created dev-board to prove design before full-size
Parts:
- removed C29, C35: 0.47uF, symbol Device:C_Small
- removed R24: 100K, symbol Device:R_Small_US
- added C20, C21: 0.1uF, symbol Device:C_Small
- added R13, R14, R15: 100K, symbol Device:R_Small_US
- C23, C25: value 0.1uF -> 0.47uF
Connections:
- net +5V is gone; now on net +3V0: C28.1, C30.1, C31.1, C32.1, C33.1, C34.1, U5.20 (PVCC), U5.29 (PVCC), U5.37 (AVCC), U5.38 (DVCC)
- net PVCC1.1 is gone; now on net +3V0: C23.1, C24.1, U4.20 (PVCC)
- net PVCC1.2 is gone; now on net +3V0: C25.1, C26.1, U4.29 (PVCC)
- net GND: now also R26.1, C20.2, C21.2, R15.1; no longer R26.2
- net INTB2: now reaches U5.45 (~{INTB})
- net INTB2: now also R14.1
- net at U5.47 (IICRST): now also R26.2; no longer R26.1
- net at U4.47 (IICRST): now also R15.2
- net INTB1: now reaches U4.45 (~{INTB})
- net INTB1: now also R13.1
- net +3.3V renamed +3V0
- net +3V0: now also C20.1, C21.1, R13.2, R14.2
- net C1.10: no longer names the net of U4.26 (CS10)
- net C1.11: no longer names the net of U4.27 (CS11)
- net C1.12: no longer names the net of U4.28 (CS12)
- net C1.13: no longer names the net of U4.30 (CS13)
- net C1.14: no longer names the net of U4.31 (CS14)
- net C1.15: no longer names the net of U4.32 (CS15)
- net C1.16: no longer names the net of U4.33 (CS16)
- net C1.4: no longer names the net of U4.19 (CS4)
- net C1.5: no longer names the net of U4.21 (CS5)
- net C1.6: no longer names the net of U4.22 (CS6)
- net C1.7: no longer names the net of U4.23 (CS7)
- net C1.8: no longer names the net of U4.24 (CS8)
- net C1.9: no longer names the net of U4.25 (CS9)
- net C2.10: no longer names the net of U5.26 (CS10)
- net C2.11: no longer names the net of U5.27 (CS11)
- net C2.12: no longer names the net of U5.28 (CS12)
- net C2.13: no longer names the net of U5.30 (CS13)
- net C2.14: no longer names the net of U5.31 (CS14)
- net C2.15: no longer names the net of U5.32 (CS15)
- net C2.4: no longer names the net of U5.19 (CS4)
- net C2.5: no longer names the net of U5.21 (CS5)
- net C2.6: no longer names the net of U5.22 (CS6)
- net C2.7: no longer names the net of U5.23 (CS7)
- net C2.8: no longer names the net of U5.24 (CS8)
- net C2.9: no longer names the net of U5.25 (CS9)
- no-connect marks 3 -> 26
Other:
- removed sheet 0
- removed sheet 1
- removed sheet 2
- removed sheet 3
- removed sheet 4
- removed sheet 5
- removed sheet 6
- removed sheet 7
- removed sheet 8
- removed sheet 9
- removed sheet A
- removed sheet Apostrophe
- removed sheet B
- removed sheet Backslash
- removed sheet Backspace
- removed sheet Bluetooth
- removed sheet Brightness
- removed sheet C
- removed sheet CAPS
- removed sheet Comma
- removed sheet D
- removed sheet DEL
- removed sheet Dash
- removed sheet Down
- removed sheet E
- removed sheet END
- removed sheet ESC
- removed sheet Enter
- removed sheet Equals
- removed sheet F
- removed sheet F1
- removed sheet F10
- removed sheet F11
- removed sheet F12
- removed sheet F2
- removed sheet F3
- removed sheet F4
- removed sheet F5
- removed sheet F6
- removed sheet F7
- removed sheet F8
- removed sheet F9
- removed sheet G
- removed sheet G1
- removed sheet G2
- removed sheet G3
- removed sheet G4
- removed sheet G5
- removed sheet GameMode
- removed sheet H
- removed sheet HOME
- removed sheet I
- removed sheet INS
- removed sheet J
- removed sheet K
- removed sheet L
- removed sheet Left
- removed sheet M
- removed sheet M1
- removed sheet M2
- removed sheet M3
- removed sheet MR
- removed sheet Menu
- removed sheet N
- removed sheet O
- removed sheet P
- removed sheet PAUSE
- removed sheet PGDN
- removed sheet PGUP
- removed sheet PRTSC
- removed sheet Period
- removed sheet Q
- removed sheet R
- removed sheet Right
- removed sheet S
- removed sheet SCRLK
- removed sheet Semicolon
- removed sheet Slash
- removed sheet Space
- removed sheet T
- removed sheet TAB
- removed sheet Tilde
- removed sheet U
- removed sheet Up
- removed sheet V
- removed sheet W
- removed sheet Wireless
- removed sheet X
- removed sheet Y
- removed sheet Z
- removed sheet lALT
- removed sheet lBracket
- removed sheet lCTRL
- removed sheet lSHIFT
- removed sheet lWIN
- removed sheet rALT
- removed sheet rBracket
- removed sheet rCTRL
- removed sheet rSHIFT
- removed sheet rWIN
- moved on the sheet: C28, C30, C31, C32, C33, C34, C36, R23, R25, R26, R27, U4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

Commit message: battery charger components
Parts:
- R13, R14, R15, R23, R25, R26, R27: footprint (none) -> keyboard:R_0402_1005Metric
Changed lines of the file:
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@@
 			)
 		)
-		(property "Footprint" ""
+		(property "Footprint" "keyboard:R_0402_1005Metric"
 			(at 219.71 120.65 0)
 			(effects
@@
 			)
 		)
-		(property "Footprint" ""
+		(property "Footprint" "keyboard:R_0402_1005Metric"
 			(at 152.4 45.72 0)
 			(effects
@@
 			)
 		)
-		(property "Footprint" ""
+		(property "Footprint" "keyboard:R_0402_1005Metric"
 			(at 152.4 57.15 0)
 			(effects
@@
 			)
 		)
-		(property "Footprint" ""
+		(property "Footprint" "keyboard:R_0402_1005Metric"
 			(at 256.54 57.15 0)
 			(effects
@@
 			)
 		)
-		(property "Footprint" ""
+		(property "Footprint" "keyboard:R_0402_1005Metric"
 			(at 227.33 120.65 0)
 			(effects
@@
 			)
 		)
-		(property "Footprint" ""
+		(property "Footprint" "keyboard:R_0402_1005Metric"
 			(at 256.54 45.72 0)
 			(effects
@@
 			)
 		)
-		(property "Footprint" ""
+		(property "Footprint" "keyboard:R_0402_1005Metric"
 			(at 187.198 118.11 0)
 			(effects
